File: kicad/FluidNC/FluidNC.kicad_pcb (KiCad board)
At the start: 2 copper layers, 210 x 120 mm, 232 parts, among them J1 USB_C_Receptacle_USB2.0, J10 Conn_01x02_Socket, J11 Conn_01x02_Socket, J12 Conn_01x02_Socket, J13 Conn_01x02_Socket, J14 Conn_01x02_Socket, J15 Conn_01x02_Socket, J16 Conn_01x12_Socket, J17 Conn_01x04_Socket, J18 Conn_01x03_Pin, J19 Conn_01x03_Pin, J20 Conn_01x04_Socket, J21 Conn_01x08_Socket, J22 Conn_01x08_Socket, J23 Conn_01x08_Socket, J24 Conn_01x08_Socket, J25 Conn_01x08_Socket, J26 Conn_01x08_Socket, J27 Conn_01x06_Pin, J31 Conn_01x02_Socket, J4 Conn_01x05_Socket, J5 Conn_01x05_Socket, J6 Conn_01x05_Socket, J7 Conn_01x05_Socket, J8 Conn_01x05_Socket, J9 Conn_01x05_Socket, Q1 BC847, Q2 BC847, SW1 SW_RESET, SW10 Macro 2, SW11 Macro 3, SW12 Resume, SW13 Pause, SW2 SW_BOOT, SW3 SW_DIP_x03, SW4 SW_DIP_x03, SW5 SW_DIP_x03, SW6 SW_DIP_x03, SW7 SW_DIP_x03, SW8 SW_DIP_x03, SW9 Macro 1, U1 CH340C, U10 ADuM120N, U11 ADuM120N, U12 LM358, U13 ADuM120N, U15 ADuM120N, U16 ADuM120N, U17 ADuM120N, U18 ADuM120N, U19 ADuM120N, U2 ESP32-WROOM-32, U21 LTV-847, U22 74HC14, U23 74HC14, U24 LTV-847, U25 LTV-847, U26 ISO1H811G, U3 74HCT595, U4 74HCT595, U5 74HCT595, U6 74HCT595, U7 ISO1H811G, U8 NCP1117-3.3_SOT223, U9 LM2596S-5

Commit message: partly route pcb
Parts:
- SW1, SW10, SW11, SW12, SW13, SW2, SW9: footprint Button_Switch_SMD:SW_SPST_B3U-1000P -> GioN_Custom:SW_SPST_B3U-1000P
- moved SW2 23.1 mm to (25.4, 60.5), turned to 90 degrees
- moved D6 9.15 mm to (114.8, 17.3)
- moved R22 5.52 mm to (114.8, 18.8)
- moved C21 3.21 mm to (57.9, 33.0)
- moved R11 3.11 mm to (66.0, 33.0)
- moved R70 3.11 mm to (85.9, 33.0)
- moved D8 3.11 mm to (89.4, 33.0)
- moved D4 3.08 mm to (69.6, 33.0)
- moved C11 2.46 mm to (110.2, 30.0), turned to -90 degrees
- moved SW1 1.69 mm to (8.13, 85.3)
- moved C12 1.27 mm to (111.2, 18.8)
- moved C72 1.14 mm to (77.7, 33.0)
- moved D5 0.92 mm to (104.6, 34.8)
- moved R62 0.52 mm to (191.0, 72.5), turned to 0 degrees
- moved R63 0.52 mm to (191.0, 67.9), turned to 0 degrees
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Routing:
- net +24V: track 146.1 -> 667.1 mm, vias 0 -> 1
- net EN_STEPPER: track 0.00 -> 179.6 mm, vias 0 -> 1
- net +5VP: track 89.0 -> 264.9 mm, vias 0 -> 2
- net GND1: track 444.2 -> 522.4 mm
- net +5V: track 42.2 -> 91.9 mm
- net GND: track 1.65 -> 44.8 mm
- net Net-(D5-K): track 0.00 -> 23.2 mm, vias 0 -> 2
- net ESP_IO0: track 26.9 -> 4.94 mm, vias 2 -> 0
- net RESUME: track 5.00 -> 23.5 mm
- net PAUSE: track 5.00 -> 23.4 mm
- net MACRO3: track 5.00 -> 23.2 mm
- net +3.3V: track 16.2 -> 32.3 mm
- net Net-(C51-Pad1): track 0.00 -> 8.23 mm
- net Net-(C48-Pad1): track 0.00 -> 8.23 mm
- net Net-(C62-Pad1): track 0.00 -> 8.18 mm
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
Commit message: Update FluidNC.kicad_pcb
Parts:
- moved C52 2.35 mm to (120.7, 62.2)
- moved C56 2.35 mm to (110.5, 62.2)
- moved C57 2.35 mm to (105.4, 62.2)
- moved R37 2.35 mm to (123.2, 62.2)
- moved R42 2.35 mm to (118.1, 62.2)
- moved R56 2.35 mm to (113.0, 62.2)
- moved R57 2.35 mm to (108.0, 62.2)
- moved C53 2.35 mm to (123.2, 65.8)
- moved C55 2.35 mm to (118.1, 65.8)
- moved C60 2.35 mm to (113.0, 65.8)
- moved C61 2.35 mm to (108.0, 65.8)
- moved R36 2.35 mm to (120.7, 65.7)
- moved R52 2.35 mm to (110.5, 65.7)
- moved R53 2.35 mm to (105.4, 65.7)
- moved C54 2.35 mm to (115.6, 62.2)
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Routing:
- net IO4_MACRO1: track 2.13 -> 207.2 mm, vias 0 -> 2
- net IO26_MACRO2: track 2.13 -> 189.8 mm, vias 0 -> 2
- net IO27_MACRO3: track 2.17 -> 166.0 mm, vias 0 -> 2
- net IO36_HOME1: track 2.19 -> 162.8 mm, vias 0 -> 2
- net IO34_HOME2: track 2.24 -> 151.6 mm, vias 0 -> 2
- net IO13_PAUSE: track 2.30 -> 147.6 mm, vias 0 -> 2
- net IO35_HOME3: track 2.24 -> 145.0 mm, vias 0 -> 2
- net IO14_RESUME: track 2.30 -> 143.7 mm, vias 0 -> 2
- net IO22_HOME4: track 2.09 -> 138.5 mm, vias 0 -> 2
- net IO39_HOME5: track 2.09 -> 127.8 mm, vias 0 -> 2
- net IO25_HOME6: track 2.09 -> 118.4 mm, vias 0 -> 2
- net +5V: track 91.9 -> 202.0 mm, vias 2 -> 14
- net MACRO1: track 7.03 -> 80.1 mm
- net ESP_EN: track 0.00 -> 72.8 mm, vias 0 -> 2
- net MACRO2: track 7.03 -> 66.8 mm
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
Commit message: update KiCad8
Parts:
- moved R24 6.18 mm to (188.5, 103.1), turned to 0 degrees
- moved R43 5.18 mm to (93.5, 103.1), turned to 0 degrees
- moved R33 4.83 mm to (159.8, 103.1), turned to 0 degrees
- moved R60 2.05 mm to (64.8, 103.1), turned to 0 degrees
- moved R61 1.33 mm to (35.6, 103.4), turned to 0 degrees
- moved R38 1.23 mm to (130.6, 103.1), turned to 0 degrees
Routing:
- net +5VP: track 264.9 -> 655.3 mm, vias 2 -> 21
- net +24V: track 667.1 -> 916.6 mm, vias 1 -> 7
- net GND: track 64.3 -> 266.3 mm, vias 1 -> 46
- net GND1: track 522.4 -> 687.6 mm, vias 0 -> 17
- net +3.3V: track 76.1 -> 224.9 mm, vias 0 -> 14
- net +5V: track 202.0 -> 346.0 mm, vias 14 -> 22
- net HOME1: track 5.00 -> 109.8 mm, vias 0 -> 2
- net HOME6: track 5.00 -> 107.7 mm, vias 0 -> 4
- net HOME5: track 5.00 -> 77.1 mm, vias 0 -> 2
- net HOME2: track 5.00 -> 64.0 mm, vias 0 -> 2
- net HOME4: track 5.00 -> 52.4 mm, vias 0 -> 2
- net HOME3: track 5.00 -> 44.9 mm, vias 0 -> 2
- net RX: track 35.1 -> 35.8 mm
- added copper zone on B.Cu, net GND
- added copper zone on F.Cu, net GND
- added copper zone on B.Cu, net GND1
- added copper zone on F.Cu, net GND1
Other:
- board text added: "+5V"
- board text added: "24V"
- board text added: "24V / 5V"
- board text added: "24V IN"
- board text added: "FluidNC Controller V2 R1 Nikos Gioulekas 05/2024"
- board text added: "GND IN"
- board text added: "MACRO 1"
- board text added: "MACRO 2"
- board text added: "MACRO 3"
- board text added: "OUT 00"
- board text added: "OUT 01"
- board text added: "OUT 02"
- board text added: "OUT 03"
- board text added: "OUT 04"
- board text added: "OUT 05"
- board text added: "OUT 06"
- board text added: "OUT 07"
- board text added: "OUT 08"
- board text added: "OUT 09"
- board text added: "OUT 10"
- board text added: "OUT 11"
- board text added: "OUT 12"
- board text added: "OUT 13"
- board text added: "OUT FLD"
- board text added: "OUT MIST"
- board text added: "PAUSE"
- board text added: "RESUM"
- board text removed: "FluidNC Controller V1 R2 Nikos Gioulekas 02/2024"

Commit message: Finish V2 R1
Parts:
- added C31: 10n, Capacitor_SMD:C_0603_1608Metric_Pad1.08x0.95mm_HandSolder, F.Cu at (52.6, 20.4)
- added C38: 10n, Capacitor_SMD:C_0603_1608Metric_Pad1.08x0.95mm_HandSolder, F.Cu at (56.1, 20.4)
- added C73: 10n, Capacitor_SMD:C_0603_1608Metric_Pad1.08x0.95mm_HandSolder, F.Cu at (59.6, 20.4)
- added C74: 10n, Capacitor_SMD:C_0603_1608Metric_Pad1.08x0.95mm_HandSolder, F.Cu at (63.1, 20.4)
- added C75: 10n, Capacitor_SMD:C_0603_1608Metric_Pad1.08x0.95mm_HandSolder, F.Cu at (66.6, 20.4)
- added C76: 10n, Capacitor_SMD:C_0603_1608Metric_Pad1.08x0.95mm_HandSolder, F.Cu at (70.1, 20.4)
- added C77: 10n, Capacitor_SMD:C_0603_1608Metric_Pad1.08x0.95mm_HandSolder, F.Cu at (73.6, 20.4)
- added C78: 10n, Capacitor_SMD:C_0603_1608Metric_Pad1.08x0.95mm_HandSolder, F.Cu at (77.1, 20.4)
- added C79: 10n, Capacitor_SMD:C_0603_1608Metric_Pad1.08x0.95mm_HandSolder, F.Cu at (83.3, 20.3)
- added C80: 10n, Capacitor_SMD:C_0603_1608Metric_Pad1.08x0.95mm_HandSolder, F.Cu at (86.8, 20.3)
- added C81: 10n, Capacitor_SMD:C_0603_1608Metric_Pad1.08x0.95mm_HandSolder, F.Cu at (90.3, 20.3)
- added C82: 10n, Capacitor_SMD:C_0603_1608Metric_Pad1.08x0.95mm_HandSolder, F.Cu at (93.8, 20.3)
- added C83: 10n, Capacitor_SMD:C_0603_1608Metric_Pad1.08x0.95mm_HandSolder, F.Cu at (97.3, 20.3)
- added C84: 10n, Capacitor_SMD:C_0603_1608Metric_Pad1.08x0.95mm_HandSolder, F.Cu at (100.8, 20.3)
- added C85: 10n, Capacitor_SMD:C_0603_1608Metric_Pad1.08x0.95mm_HandSolder, F.Cu at (104.3, 20.3)
- added C86: 10n, Capacitor_SMD:C_0603_1608Metric_Pad1.08x0.95mm_HandSolder, F.Cu at (107.8, 20.3)
- added D11: LED, LED_SMD:LED_0603_1608Metric_Pad1.05x0.95mm_HandSolder, F.Cu at (52.6, 17.2)
- added D12: LED, LED_SMD:LED_0603_1608Metric_Pad1.05x0.95mm_HandSolder, F.Cu at (56.1, 17.2)
- added D13: LED, LED_SMD:LED_0603_1608Metric_Pad1.05x0.95mm_HandSolder, F.Cu at (59.6, 17.2)
- added D14: LED, LED_SMD:LED_0603_1608Metric_Pad1.05x0.95mm_HandSolder, F.Cu at (63.1, 17.2)
- added D15: LED, LED_SMD:LED_0603_1608Metric_Pad1.05x0.95mm_HandSolder, F.Cu at (66.6, 17.2)
- added D16: LED, LED_SMD:LED_0603_1608Metric_Pad1.05x0.95mm_HandSolder, F.Cu at (70.1, 17.2)
- added D17: LED, LED_SMD:LED_0603_1608Metric_Pad1.05x0.95mm_HandSolder, F.Cu at (73.6, 17.2)
- added D18: LED, LED_SMD:LED_0603_1608Metric_Pad1.05x0.95mm_HandSolder, F.Cu at (77.1, 17.2)
- added D19: LED, LED_SMD:LED_0603_1608Metric_Pad1.05x0.95mm_HandSolder, F.Cu at (83.3, 17.1)
- added D20: LED, LED_SMD:LED_0603_1608Metric_Pad1.05x0.95mm_HandSolder, F.Cu at (86.8, 17.1)
- added D21: LED, LED_SMD:LED_0603_1608Metric_Pad1.05x0.95mm_HandSolder, F.Cu at (90.3, 17.1)
- added D22: LED, LED_SMD:LED_0603_1608Metric_Pad1.05x0.95mm_HandSolder, F.Cu at (93.8, 17.1)
- added D23: LED, LED_SMD:LED_0603_1608Metric_Pad1.05x0.95mm_HandSolder, F.Cu at (97.3, 17.1)
- added D24: LED, LED_SMD:LED_0603_1608Metric_Pad1.05x0.95mm_HandSolder, F.Cu at (100.8, 17.1)
- added D25: LED, LED_SMD:LED_0603_1608Metric_Pad1.05x0.95mm_HandSolder, F.Cu at (104.3, 17.1)
- added D26: LED, LED_SMD:LED_0603_1608Metric_Pad1.05x0.95mm_HandSolder, F.Cu at (107.8, 17.1)
- added D27: LED, LED_SMD:LED_0603_1608Metric_Pad1.05x0.95mm_HandSolder, F.Cu at (24.6, 26.1)
- added D28: LED, LED_SMD:LED_0603_1608Metric_Pad1.05x0.95mm_HandSolder, F.Cu at (47.0, 23.5)
- added D29: LED, LED_SMD:LED_0603_1608Metric_Pad1.05x0.95mm_HandSolder, F.Cu at (175.8, 103.2)
- added D30: LED, LED_SMD:LED_0603_1608Metric_Pad1.05x0.95mm_HandSolder, F.Cu at (146.7, 103.6)
- added D31: LED, LED_SMD:LED_0603_1608Metric_Pad1.05x0.95mm_HandSolder, F.Cu at (117.9, 103.6)
- added D32: LED, LED_SMD:LED_0603_1608Metric_Pad1.05x0.95mm_HandSolder, F.Cu at (80.7, 103.6)
- added D33: LED, LED_SMD:LED_0603_1608Metric_Pad1.05x0.95mm_HandSolder, F.Cu at (51.8, 103.6)
- added D34: LED, LED_SMD:LED_0603_1608Metric_Pad1.05x0.95mm_HandSolder, F.Cu at (23.0, 103.6)
- added D35: LED, LED_SMD:LED_0603_1608Metric_Pad1.05x0.95mm_HandSolder, F.Cu at (186.1, 47.7)
- added D36: LED, LED_SMD:LED_0603_1608Metric_Pad1.05x0.95mm_HandSolder, F.Cu at (186.1, 46.0)
- added D37: LED, LED_SMD:LED_0603_1608Metric_Pad1.05x0.95mm_HandSolder, F.Cu at (186.1, 44.3)
- added D38: LED, LED_SMD:LED_0603_1608Metric_Pad1.05x0.95mm_HandSolder, F.Cu at (186.1, 42.6)
- added D39: LED, LED_SMD:LED_0603_1608Metric_Pad1.05x0.95mm_HandSolder, F.Cu at (186.1, 40.9)
- added R100: 10k, Resistor_SMD:R_0603_1608Metric_Pad0.98x0.95mm_HandSolder, F.Cu at (121.5, 103.6)
- added R101: 10k, Resistor_SMD:R_0603_1608Metric_Pad0.98x0.95mm_HandSolder, F.Cu at (84.2, 103.6)
- added R102: 10k, Resistor_SMD:R_0603_1608Metric_Pad0.98x0.95mm_HandSolder, F.Cu at (55.3, 103.6)
- added R103: 10k, Resistor_SMD:R_0603_1608Metric_Pad0.98x0.95mm_HandSolder, F.Cu at (26.5, 103.6)
- added R104: 10k, Resistor_SMD:R_0603_1608Metric_Pad0.98x0.95mm_HandSolder, F.Cu at (182.6, 47.7)
- added R105: 10k, Resistor_SMD:R_0603_1608Metric_Pad0.98x0.95mm_HandSolder, F.Cu at (182.6, 46.0)
- added R106: 10k, Resistor_SMD:R_0603_1608Metric_Pad0.98x0.95mm_HandSolder, F.Cu at (182.6, 44.3)
- added R107: 10k, Resistor_SMD:R_0603_1608Metric_Pad0.98x0.95mm_HandSolder, F.Cu at (182.6, 42.6)
- added R108: 10k, Resistor_SMD:R_0603_1608Metric_Pad0.98x0.95mm_HandSolder, F.Cu at (182.6, 40.9)
- added R71: 10k, Resistor_SMD:R_0603_1608Metric_Pad0.98x0.95mm_HandSolder, F.Cu at (52.6, 18.8)
- added R75: 10k, Resistor_SMD:R_0603_1608Metric_Pad0.98x0.95mm_HandSolder, F.Cu at (56.1, 18.8)
- added R79: 10k, Resistor_SMD:R_0603_1608Metric_Pad0.98x0.95mm_HandSolder, F.Cu at (59.6, 18.8)
- added R83: 10k, Resistor_SMD:R_0603_1608Metric_Pad0.98x0.95mm_HandSolder, F.Cu at (63.1, 18.8)
- added R84: 10k, Resistor_SMD:R_0603_1608Metric_Pad0.98x0.95mm_HandSolder, F.Cu at (66.6, 18.8)
- added R85: 10k, Resistor_SMD:R_0603_1608Metric_Pad0.98x0.95mm_HandSolder, F.Cu at (70.1, 18.8)
- added R86: 10k, Resistor_SMD:R_0603_1608Metric_Pad0.98x0.95mm_HandSolder, F.Cu at (73.6, 18.8)
- added R87: 10k, Resistor_SMD:R_0603_1608Metric_Pad0.98x0.95mm_HandSolder, F.Cu at (77.1, 18.8)
- added R88: 10k, Resistor_SMD:R_0603_1608Metric_Pad0.98x0.95mm_HandSolder, F.Cu at (83.3, 18.7)
- added R89: 10k, Resistor_SMD:R_0603_1608Metric_Pad0.98x0.95mm_HandSolder, F.Cu at (86.8, 18.7)
- added R90: 10k, Resistor_SMD:R_0603_1608Metric_Pad0.98x0.95mm_HandSolder, F.Cu at (90.3, 18.7)
- added R91: 10k, Resistor_SMD:R_0603_1608Metric_Pad0.98x0.95mm_HandSolder, F.Cu at (93.8, 18.7)
- added R92: 10k, Resistor_SMD:R_0603_1608Metric_Pad0.98x0.95mm_HandSolder, F.Cu at (97.3, 18.7)
- added R93: 10k, Resistor_SMD:R_0603_1608Metric_Pad0.98x0.95mm_HandSolder, F.Cu at (100.8, 18.7)
- added R94: 10k, Resistor_SMD:R_0603_1608Metric_Pad0.98x0.95mm_HandSolder, F.Cu at (104.3, 18.7)
- added R95: 10k, Resistor_SMD:R_0603_1608Metric_Pad0.98x0.95mm_HandSolder, F.Cu at (107.8, 18.7)
- added R96: 10k, Resistor_SMD:R_0603_1608Metric_Pad0.98x0.95mm_HandSolder, F.Cu at (24.7, 24.5)
- added R97: 10k, Resistor_SMD:R_0603_1608Metric_Pad0.98x0.95mm_HandSolder, F.Cu at (47.0, 25.1)
- added R98: 10k, Resistor_SMD:R_0603_1608Metric_Pad0.98x0.95mm_HandSolder, F.Cu at (179.3, 103.2)
- added R99: 10k, Resistor_SMD:R_0603_1608Metric_Pad0.98x0.95mm_HandSolder, F.Cu at (150.2, 103.6)
- R24: value 1k5 -> 5k6
- moved L1 17.9 mm to (131.2, 26.3)
- moved U9 17.3 mm to (116.4, 25.6)
- moved D5 9.80 mm to (114.2, 37.0)
- moved C10 9.05 mm to (125.2, 37.5)
- moved F1 8.12 mm to (134.1, 35.6)
- moved C21 7.09 mm to (57.9, 40.1)
- moved C72 7.09 mm to (77.7, 40.1)
- moved D4 7.09 mm to (69.6, 40.1)
- moved D8 7.09 mm to (89.4, 40.1)
- moved R11 7.09 mm to (66.0, 40.1)
- moved R70 7.09 mm to (85.9, 40.1)
- moved U26 7.09 mm to (81.8, 31.5)
- moved U7 7.09 mm to (62.1, 31.5)
- moved C12 6.91 mm to (118.0, 18.2)
- moved D6 6.91 mm to (121.7, 16.7)
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Connections:
- J10 pad 2: GND1 -> +24V
- J11 pad 2: GND1 -> +24V
- J12 pad 2: GND1 -> +24V
- J13 pad 2: GND1 -> +24V
- J14 pad 2: GND1 -> +24V
- J15 pad 2: GND1 -> +24V
- J16 pad 2: GND1 -> +24V
- J16 pad 4: GND1 -> +24V
- J16 pad 6: GND1 -> +24V
- J16 pad 8: GND1 -> +24V
- R24 pad 2: +24V -> Net-(R24-Pad2)
- R33 pad 2: +24V -> Net-(R33-Pad2)
- R38 pad 2: +24V -> Net-(R38-Pad2)
- R43 pad 2: +24V -> Net-(R43-Pad2)
- R60 pad 2: +24V -> Net-(R60-Pad2)
- R61 pad 2: +24V -> Net-(R61-Pad2)
- R62 pad 2: +24V -> Net-(R62-Pad2)
- R63 pad 2: +24V -> Net-(R63-Pad2)
- R80 pad 2: +24V -> Net-(R80-Pad2)
- R81 pad 2: +24V -> Net-(R81-Pad2)
- R82 pad 2: +24V -> Net-(R82-Pad2)
- U21 pad 1: MACRO3 -> Net-(R80-Pad2)
- U21 pad 3: PAUSE -> Net-(R81-Pad2)
- U21 pad 5: RESUME -> Net-(R82-Pad2)
- U24 pad 1: HOME6 -> Net-(R61-Pad2)
- U24 pad 3: HOME5 -> Net-(R60-Pad2)
- U24 pad 5: HOME4 -> Net-(R43-Pad2)
- U24 pad 7: HOME3 -> Net-(R38-Pad2)
- U25 pad 1: HOME2 -> Net-(R33-Pad2)
- U25 pad 3: HOME1 -> Net-(R24-Pad2)
- U25 pad 5: MACRO1 -> Net-(R62-Pad2)
- U25 pad 7: MACRO2 -> Net-(R63-Pad2)
Routing:
- net Net-(R61-Pad2): track 0.00 -> 100.0 mm, vias 0 -> 4
- net Net-(R24-Pad2): track 0.00 -> 98.6 mm, vias 0 -> 2
- net HOME1: track 109.8 -> 16.4 mm, vias 2 -> 0
- net HOME6: track 107.7 -> 15.4 mm, vias 4 -> 0
- net Net-(R60-Pad2): track 0.00 -> 69.1 mm, vias 0 -> 2
- net Net-(R62-Pad2): track 0.00 -> 65.6 mm
- net Net-(R63-Pad2): track 0.00 -> 61.7 mm
- net HOME5: track 77.1 -> 15.9 mm, vias 2 -> 0
- net GND1: track 687.6 -> 747.2 mm, vias 17 -> 35
- net Net-(R33-Pad2): track 0.00 -> 53.9 mm, vias 0 -> 2
- net HOME2: track 64.0 -> 16.0 mm, vias 2 -> 0
- net Net-(R43-Pad2): track 0.00 -> 41.2 mm, vias 0 -> 2
- net Net-(R38-Pad2): track 0.00 -> 37.7 mm, vias 0 -> 2
- net HOME4: track 52.4 -> 15.8 mm, vias 2 -> 0
- net Net-(D25-A): track 31.4 -> 61.2 mm
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Other:
- outline, holes or cut-outs redrawn
- board text added: "RESUME"

Commit message: Add V2R1
Routing:
- net GND: track 266.3 -> 252.0 mm
- net +5V: track 346.0 -> 338.9 mm
- net I2SO23_USEROUT8: track 34.3 -> 27.3 mm
- net I2SO24_USEROUT9: track 21.7 -> 14.6 mm
- net I2SO28_USEROUT13: track 29.4 -> 22.3 mm
- net I2SO27_USEROUT12: track 29.8 -> 22.7 mm
- net I2SO26_USEROUT11: track 30.5 -> 23.4 mm
- net I2SO25_USEROUT10: track 31.2 -> 24.1 mm
- net I2SO22_USEROUT7: track 35.0 -> 27.9 mm
- net I2SO21_USEROUT6: track 35.7 -> 28.6 mm
- net GND1: track 747.2 -> 745.3 mm, vias 35 -> 34
Other:
- board text added: "DIR"
- board text added: "STEP"
