File: kicad/FluidNC/FluidNC.kicad_pcb (KiCad board)
At the start: 2 copper layers, 210 x 120 mm, 306 parts, among them J1 USB_C_Receptacle_USB2.0, J10 Conn_01x02_Socket, J11 Conn_01x02_Socket, J12 Conn_01x02_Socket, J13 Conn_01x02_Socket, J14 Conn_01x02_Socket, J15 Conn_01x02_Socket, J16 Conn_01x12_Socket, J17 Conn_01x04_Socket, J18 Conn_01x03_Pin, J19 Conn_01x03_Pin, J20 Conn_01x04_Socket, J21 Conn_01x08_Socket, J22 Conn_01x08_Socket, J23 Conn_01x08_Socket, J24 Conn_01x08_Socket, J25 Conn_01x08_Socket, J26 Conn_01x08_Socket, J27 Conn_01x06_Pin, J31 Conn_01x02_Socket, J4 Conn_01x05_Socket, J5 Conn_01x05_Socket, J6 Conn_01x05_Socket, J7 Conn_01x05_Socket, J8 Conn_01x05_Socket, J9 Conn_01x05_Socket, Q1 BC847, Q2 BC847, SW1 SW_RESET, SW10 Macro 2, SW11 Macro 3, SW12 Resume, SW13 Pause, SW2 SW_BOOT, SW3 SW_DIP_x03, SW4 SW_DIP_x03, SW5 SW_DIP_x03, SW6 SW_DIP_x03, SW7 SW_DIP_x03, SW8 SW_DIP_x03, SW9 Macro 1, U1 CH340C, U10 ADuM120N, U11 ADuM120N, U12 LM358, U13 ADuM120N, U15 ADuM120N, U16 ADuM120N, U17 ADuM120N, U18 ADuM120N, U19 ADuM120N, U2 ESP32-WROOM-32, U21 LTV-847, U22 74HC14, U23 74HC14, U24 LTV-847, U25 LTV-847, U26 ISO1H811G, U3 74HCT595, U4 74HCT595, U5 74HCT595, U6 74HCT595, U7 ISO1H811G, U8 NCP1117-3.3_SOT223, U9 LM2596S-5

Commit message: Add debug features
Change PCB Color
Add ground pins for probing
Add debug leds for step, dir and stepper_en
Add silkscreen with pin definitions
Parts:
- added D40: LED, LED_SMD:LED_0603_1608Metric_Pad1.05x0.95mm_HandSolder, F.Cu at (80.3, 70.7)
- added D41: LED, LED_SMD:LED_0603_1608Metric_Pad1.05x0.95mm_HandSolder, F.Cu at (81.8, 70.7)
- added D42: LED, LED_SMD:LED_0603_1608Metric_Pad1.05x0.95mm_HandSolder, F.Cu at (83.3, 70.7)
- added D43: LED, LED_SMD:LED_0603_1608Metric_Pad1.05x0.95mm_HandSolder, F.Cu at (84.8, 70.7)
- added D44: LED, LED_SMD:LED_0603_1608Metric_Pad1.05x0.95mm_HandSolder, F.Cu at (86.4, 70.7)
- added D45: LED, LED_SMD:LED_0603_1608Metric_Pad1.05x0.95mm_HandSolder, F.Cu at (87.9, 70.7)
- added D46: LED, LED_SMD:LED_0603_1608Metric_Pad1.05x0.95mm_HandSolder, F.Cu at (89.4, 70.7)
- added D47: LED, LED_SMD:LED_0603_1608Metric_Pad1.05x0.95mm_HandSolder, F.Cu at (90.9, 70.7)
- added D48: LED, LED_SMD:LED_0603_1608Metric_Pad1.05x0.95mm_HandSolder, F.Cu at (92.5, 70.7)
- added D49: LED, LED_SMD:LED_0603_1608Metric_Pad1.05x0.95mm_HandSolder, F.Cu at (94.0, 70.7)
- added D50: LED, LED_SMD:LED_0603_1608Metric_Pad1.05x0.95mm_HandSolder, F.Cu at (95.5, 70.7)
- added D51: LED, LED_SMD:LED_0603_1608Metric_Pad1.05x0.95mm_HandSolder, F.Cu at (97.0, 70.7)
- added D52: LED, LED_SMD:LED_0603_1608Metric_Pad1.05x0.95mm_HandSolder, F.Cu at (99.2, 70.7)
- added J2: Conn_01x01_Pin, Connector_PinHeader_2.54mm:PinHeader_1x01_P2.54mm_Vertical, F.Cu at (44.3, 43.5)
- added J28: Conn_01x01_Pin, Connector_PinHeader_2.54mm:PinHeader_1x01_P2.54mm_Vertical, F.Cu at (96.7, 56.7)
- added J29: Conn_01x01_Pin, Connector_PinHeader_2.54mm:PinHeader_1x01_P2.54mm_Vertical, F.Cu at (191.0, 38.4)
- added J3: Conn_01x01_Pin, Connector_PinHeader_2.54mm:PinHeader_1x01_P2.54mm_Vertical, F.Cu at (167.6, 48.9)
- added J30: Conn_01x01_Pin, Connector_PinHeader_2.54mm:PinHeader_1x01_P2.54mm_Vertical, F.Cu at (100.5, 106.5)
- added J32: Conn_01x01_Pin, Connector_PinHeader_2.54mm:PinHeader_1x01_P2.54mm_Vertical, F.Cu at (105.9, 27.5)
- added R109: 10k, Resistor_SMD:R_0603_1608Metric_Pad0.98x0.95mm_HandSolder, F.Cu at (80.3, 67.3)
- added R110: 10k, Resistor_SMD:R_0603_1608Metric_Pad0.98x0.95mm_HandSolder, F.Cu at (81.8, 67.3)
- added R111: 10k, Resistor_SMD:R_0603_1608Metric_Pad0.98x0.95mm_HandSolder, F.Cu at (83.3, 67.3)
- added R112: 10k, Resistor_SMD:R_0603_1608Metric_Pad0.98x0.95mm_HandSolder, F.Cu at (84.8, 67.3)
- added R113: 10k, Resistor_SMD:R_0603_1608Metric_Pad0.98x0.95mm_HandSolder, F.Cu at (86.4, 67.3)
- added R114: 10k, Resistor_SMD:R_0603_1608Metric_Pad0.98x0.95mm_HandSolder, F.Cu at (87.9, 67.3)
- added R115: 10k, Resistor_SMD:R_0603_1608Metric_Pad0.98x0.95mm_HandSolder, F.Cu at (89.4, 67.3)
- added R116: 10k, Resistor_SMD:R_0603_1608Metric_Pad0.98x0.95mm_HandSolder, F.Cu at (90.9, 67.3)
- added R117: 10k, Resistor_SMD:R_0603_1608Metric_Pad0.98x0.95mm_HandSolder, F.Cu at (92.5, 67.3)
- added R118: 10k, Resistor_SMD:R_0603_1608Metric_Pad0.98x0.95mm_HandSolder, F.Cu at (94.0, 67.3)
- added R119: 10k, Resistor_SMD:R_0603_1608Metric_Pad0.98x0.95mm_HandSolder, F.Cu at (95.5, 67.3)
- added R120: 10k, Resistor_SMD:R_0603_1608Metric_Pad0.98x0.95mm_HandSolder, F.Cu at (97.0, 67.3)
- added R121: 10k, Resistor_SMD:R_0603_1608Metric_Pad0.98x0.95mm_HandSolder, F.Cu at (99.2, 67.3)
Routing:
- net I2SO8_DIR2: track 27.1 -> 75.2 mm, vias 0 -> 2
- net I2SO10_DIR1: track 26.4 -> 74.0 mm, vias 0 -> 2
- net I2SO9_STEP2: track 21.3 -> 68.5 mm, vias 0 -> 2
- net I2SO3_STEP5: track 14.7 -> 61.3 mm, vias 0 -> 2
- net I2SO2_DIR5: track 14.7 -> 61.0 mm, vias 0 -> 2
- net I2SO7_STEP3: track 20.6 -> 66.6 mm, vias 0 -> 2
- net I2SO11_STEP1: track 26.7 -> 72.6 mm, vias 0 -> 2
- net I2SO0_DIR6: track 23.7 -> 69.3 mm, vias 0 -> 2
- net I2SO1_STEP6: track 17.5 -> 63.0 mm, vias 0 -> 2
- net I2SO5_STEP4: track 15.4 -> 59.5 mm, vias 0 -> 2
- net I2SO4_DIR4: track 15.4 -> 59.1 mm, vias 0 -> 2
- net I2SO6_DIR3: track 21.2 -> 61.4 mm, vias 0 -> 2
- net I2SO14_EN_STEPPER: track 29.8 -> 57.2 mm
- net GND: track 252.0 -> 248.1 mm, vias 46 -> 47
- net Net-(D52-A): track 0.00 -> 1.64 mm
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Other:
- outline, holes or cut-outs redrawn
- board text added: "DIR1"
- board text added: "DIR2"
- board text added: "DIR3"
- board text added: "DIR4"
- board text added: "DIR5"
- board text added: "DIR6"
- board text added: "PGND"
- board text added: "PIN Definitions: I2SO.00 -> DIR 6 I2SO.01 -> STEP 6 I2SO.02 -> DIR 5 I2SO.03 -> STEP 5 I2SO.04 -> DIR 4 I2SO.05 -> STEP 4 I2SO.06 -> DIR 3 I2SO.07 -> STEP 3 I2SO.08 -> DIR 2 I2SO.09 -> STEP 2 I2SO.10 -> DIR 1 I2SO.11 -> STEP 1 I2SO.12 -> MIST I2SO.13 -> FLOOD I2SO.14 -> EN STEPPER I2SO.15 -> USER 0 I2SO.16 -> USER 1 I2SO.17 -> USER 2 I2SO.18 -> USER 3 I2SO.19 -> USER 4 I2SO.20 -> USER 5 I2SO.21 -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"
- board text added: "PIN Definitions: OUTPUTS: IO32 -> PWM 1 IO33 -> PWM 2 INPUTS: IO36 -> HOME 1 IO34 -> HOME 2 IO35 -> HOME 3 IO22 -> HOME 4 IO39 -> HOME 5 IO25 -> HOME 6 IO04 -> MACRO 1 IO26 -> MACRO 2 IO27 -> MACRO 3 IO13 -> PAUSE IO14 -> RESUME DIGITAL (I2SO): IO21 -> I2SO DATA IO16 -> I2SO BCK IO17 -> I2SO WS J27: +5V -> PIN 1 IO05 -> PIN 2 (SPI CS) IO18 -> PIN 3 (SPI SCK) IO19 -> PIN 4 (SPI MISO) IO23 -> PIN 5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"
- board text added: "STEP1"
- board text added: "STEP2"
- board text added: "STEP3"
- board text added: "STEP4"
- board text added: "STEP5"
- board text added: "STEP6"
- board text added: "STEPPER ENABLE"

Commit message: Update FluidNC.kicad_pcb
Other:
- board text added: "FluidNC Controller V2 R2 Nikos Gioulekas 05/2024"
- board text removed: "FluidNC Controller V2 R1 Nikos Gioulekas 05/2024"
Changed lines of the file:
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@@
 		(tags "THT DIP DIL PDIP 2.54mm 8.89mm 350mil SMDSocket LongPads")
 		(property "Reference" "U25"
-			(at 0.254 -8.934 90)
+			(at -0.005 11.41 90)
 			(layer "F.SilkS")
 			(effects
@@
 		)
 	)
-	(gr_text "FluidNC Controller V2 R1\nNikos Gioulekas\n05/2024"
+	(gr_text "FluidNC Controller V2 R2\nNikos Gioulekas\n05/2024"
 		(at 158.7 39.8 0)
 		(layer "F.SilkS")
