File: kicad/FluidNC/FluidNC.kicad_pcb (KiCad board)
At the start: 2 copper layers, 210 x 120 mm, 338 parts, among them J1 USB_C_Receptacle_USB2.0, J10 Conn_01x02_Socket, J11 Conn_01x02_Socket, J12 Conn_01x02_Socket, J13 Conn_01x02_Socket, J14 Conn_01x02_Socket, J15 Conn_01x02_Socket, J16 Conn_01x12_Socket, J17 Conn_01x04_Socket, J18 Conn_01x03_Pin, J19 Conn_01x03_Pin, J2 Conn_01x01_Pin, J20 Conn_01x04_Socket, J21 Conn_01x08_Socket, J22 Conn_01x08_Socket, J23 Conn_01x08_Socket, J24 Conn_01x08_Socket, J25 Conn_01x08_Socket, J26 Conn_01x08_Socket, J27 Conn_01x06_Pin, J28 Conn_01x01_Pin, J29 Conn_01x01_Pin, J3 Conn_01x01_Pin, J30 Conn_01x01_Pin, J31 Conn_01x02_Socket, J32 Conn_01x01_Pin, J4 Conn_01x05_Socket, J5 Conn_01x05_Socket, J6 Conn_01x05_Socket, J7 Conn_01x05_Socket, J8 Conn_01x05_Socket, J9 Conn_01x05_Socket, Q1 BC847, Q2 BC847, SW1 SW_RESET, SW10 Macro 2, SW11 Macro 3, SW12 Resume, SW13 Pause, SW2 SW_BOOT, SW3 SW_DIP_x03, SW4 SW_DIP_x03, SW5 SW_DIP_x03, SW6 SW_DIP_x03, SW7 SW_DIP_x03, SW8 SW_DIP_x03, SW9 Macro 1, U1 CH340C, U10 ADuM120N, U11 ADuM120N, U12 LM358, U13 ADuM120N, U15 ADuM120N, U16 ADuM120N, U17 ADuM120N, U18 ADuM120N, U19 ADuM120N, U2 ESP32-WROOM-32, U21 LTV-847, U22 74HC14, U23 74HC14, U24 LTV-847, U25 LTV-847, U26 ISO1H811G, U3 74HCT595, U4 74HCT595, U5 74HCT595, U6 74HCT595, U7 ISO1H811G, U8 NCP1117-3.3_SOT223, U9 LM2596S-5

Commit message: Update schematic
Remove 1N4148 in PWM to 10V converter, connect test input buttons to 24V instead of ground, tune some resistors and caps
Parts:
- removed D10, D9: 1N4148WS, Diode_SMD:D_SOD-323
- C23, C24: value 1u -> 100n
- D11, D12, D13, D14, D15, D16, D17, D18, D19, D20, D21, D22, D23, D24, D25, D26, D27, D28, D4, D40, D41, D42, D43, D44, D45, D46, D47, D48, D49, D50, D51, D52, D8: value LED -> rt
- D2, D3: value LED -> bl
- D29, D30, D31, D32, D33, D34, D35, D36, D37, D38, D39: value LED -> ye
- D6, D7: value LED -> gn
- R13, R18: value 100R -> 10k
- R96, R97: value 10k -> 5k1
Connections:
- R13 pad 1: Net-(D9-K) -> PWM1
- R14 pad 1: Net-(D9-K) -> PWM1
- R17 pad 1: Net-(D10-K) -> PWM2
- R18 pad 1: Net-(D10-K) -> PWM2
- SW10 pad 2: GND1 -> +24V
- SW11 pad 2: GND1 -> +24V
- SW12 pad 2: GND1 -> +24V
- SW13 pad 2: GND1 -> +24V
- SW9 pad 2: GND1 -> +24V
Routing:
- net +24V: track 922.8 -> 973.0 mm, vias 3 -> 6
- net GND1: track 745.3 -> 752.9 mm
- net PWM2: track 43.5 -> 47.5 mm
- net Net-(D9-K): track 3.85 -> 0.00 mm
- net Net-(D10-K): track 3.67 -> 0.00 mm

Commit message: Update FluidNC.kicad_pcb
Parts:
- moved C30 1.13 mm to (56.1, 77.9)
- moved C35 0.98 mm to (49.1, 77.9)
- moved U19 0.81 mm to (31.6, 73.4)
- moved C29 0.52 mm to (56.1, 68.6)
- moved C36 0.50 mm to (42.0, 77.9)
- moved C32 0.41 mm to (49.1, 68.6)
- moved C34 0.38 mm to (35.1, 68.6)
- moved U18 0.34 mm to (38.6, 73.4)
- moved U16 0.33 mm to (52.6, 73.4)
- moved U17 0.31 mm to (45.6, 73.4)
- moved C13 0.25 mm to (76.7, 68.6)
- moved C25 0.24 mm to (69.9, 68.6)
- moved C27 0.23 mm to (63.1, 68.6)
- moved C37 0.11 mm to (35.2, 77.9)
- moved C26 0.08 mm to (70.0, 78.0)
Routing:
- net GND1: track 752.9 -> 759.8 mm
- net GND: track 248.1 -> 250.0 mm
- net +5VP: track 675.0 -> 676.1 mm
- net STEP6: track 28.1 -> 27.3 mm
- net +3.3V: track 224.9 -> 225.7 mm
- net IO33_PWM2: track 64.5 -> 65.1 mm
- net I2SO0_DIR6: track 69.3 -> 69.8 mm
- net I2SO1_STEP6: track 63.0 -> 63.5 mm

Commit message: Minor changes
Add designated 3.2mm hole footprints,
update packages
Parts:
- added M3: MountingHole_3.2mm_M3_Pad_Via, MountingHole:MountingHole_3.2mm_M3_Pad_Via, F.Cu at (5.00, 5.00)
- added M3: MountingHole_3.2mm_M3_Pad_Via, MountingHole:MountingHole_3.2mm_M3_Pad_Via, F.Cu at (100.0, 115.0)
- added M3: MountingHole_3.2mm_M3_Pad_Via, MountingHole:MountingHole_3.2mm_M3_Pad_Via, F.Cu at (131.5, 18.7)
- added M3: MountingHole_3.2mm_M3_Pad_Via, MountingHole:MountingHole_3.2mm_M3_Pad_Via, F.Cu at (5.00, 115.0)
- added M3: MountingHole_3.2mm_M3_Pad_Via, MountingHole:MountingHole_3.2mm_M3_Pad_Via, F.Cu at (205.0, 5.00)
- added M3: MountingHole_3.2mm_M3_Pad_Via, MountingHole:MountingHole_3.2mm_M3_Pad_Via, F.Cu at (205.0, 115.0)
- C42, C43, C44, C45, C46, C47: footprint Capacitor_SMD:CP_Elec_10x7.9 -> Capacitor_SMD:CP_Elec_8x10.5
- D1: footprint Diode_SMD:D_SOD-323 -> Diode_SMD:D_SOD-323_HandSoldering
- D5: value D_Schottky -> SS34; footprint Diode_SMD:D_SMC -> Diode_SMD:D_SMA
- L1: footprint Inductor_SMD:L_7.3x7.3_H3.5 -> Inductor_SMD:L_6.3x6.3_H3
- moved C45 0.32 mm to (134.6, 93.7)
- moved C46 0.32 mm to (166.6, 93.7)
- moved C44 0.31 mm to (102.6, 93.7)
- moved C42 0.10 mm to (38.1, 93.7)
Routing:
- net +5VP: track 676.1 -> 671.1 mm
- net +24V: track 973.0 -> 977.8 mm
- net Net-(J31-Pin_1): track 29.7 -> 32.5 mm
- net TX: track 32.0 -> 31.2 mm
Other:
- outline, holes or cut-outs redrawn
- board text added: "ENA"
