File: kicad/FluidNC/inputs.kicad_sch (KiCad schematic)
At the start: 96 parts, among them J10 Conn_01x02_Socket, J11 Conn_01x02_Socket, J12 Conn_01x02_Socket, J13 Conn_01x02_Socket, J14 Conn_01x02_Socket, J15 Conn_01x02_Socket, J16 Conn_01x12_Socket, SW1 Macro 1, SW1 Macro 2, SW1 Macro 3, SW1 Pause, SW1 Resume, U21 LTV-847, U22 74HC14, U23 74HC14, U24 LTV-847, U25 LTV-847

Commit message: USB-C CC fix
Parts:
- renumbered C5 to C48, C5 to C49, C5 to C50, C5 to C51, C5 to C52, C5 to C53, C5 to C54, C5 to C55, C5 to C56, C5 to C57, C5 to C58, C5 to C59, C5 to C60, C5 to C61, C5 to C62, C5 to C63, C5 to C64, C5 to C65, C5 to C66, C5 to C67, C5 to C68, C5 to C69, C5 to C70, C5 to C71, R3 to R24, R3 to R25, R3 to R26, R3 to R27, R3 to R28, R3 to R29, R3 to R30, R3 to R31, R3 to R32, R3 to R33, R3 to R34, R3 to R35, R3 to R36, R3 to R37, R3 to R38, R3 to R39, R3 to R40, R3 to R41, R3 to R42, R3 to R43, R3 to R44, R3 to R45, R3 to R46, R3 to R47, R3 to R48, R3 to R49, R3 to R50, R3 to R51, R3 to R52, R3 to R53, R3 to R54, R3 to R55, R3 to R56, R3 to R57, R3 to R58, R3 to R59, R3 to R60, R3 to R61, R3 to R62, R3 to R63, R3 to R64, R3 to R65, R3 to R66, R3 to R67, R3 to R68, R3 to R69, R3 to R72, R3 to R73, R3 to R74, R3 to R76, R3 to R77, R3 to R78, R3 to R80, R3 to R81, R3 to R82, SW1 to SW10, SW1 to SW11, SW1 to SW12, SW1 to SW13, SW1 to SW9

Commit message: Update schematic
reduce size, changed connectors, improoved schematic
Parts:
- J10, J11, J12, J13, J14, J15: footprint GioN_Custom:TerminalBlock_WAGO_236-402_1x02_P5.00mm_45Degree -> GioN_Custom:WAGO_250-202_1x02_P3.50mm
- J16: footprint GioN_Custom:TerminalBlock_WAGO_236-412_1x12_P5.00mm_45Degree -> GioN_Custom:WAGO_250-212_1x12_P3.50mm
Changed lines of the file:
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@@
       (effects (font (size 1.27 1.27)) (justify left))
     )
-    (property "Footprint" "GioN_Custom:TerminalBlock_WAGO_236-402_1x02_P5.00mm_45Degree" (at 347.98 19.05 0)
+    (property "Footprint" "GioN_Custom:WAGO_250-202_1x02_P3.50mm" (at 347.98 19.05 0)
       (effects (font (size 1.27 1.27)) hide)
     )
@@
       (effects (font (size 1.27 1.27)) (justify left))
     )
-    (property "Footprint" "GioN_Custom:TerminalBlock_WAGO_236-402_1x02_P5.00mm_45Degree" (at 347.98 82.55 0)
+    (property "Footprint" "GioN_Custom:WAGO_250-202_1x02_P3.50mm" (at 347.98 82.55 0)
       (effects (font (size 1.27 1.27)) hide)
     )
@@
       (effects (font (size 1.27 1.27)) (justify left))
     )
-    (property "Footprint" "GioN_Custom:TerminalBlock_WAGO_236-402_1x02_P5.00mm_45Degree" (at 347.98 57.15 0)
+    (property "Footprint" "GioN_Custom:WAGO_250-202_1x02_P3.50mm" (at 347.98 57.15 0)
       (effects (font (size 1.27 1.27)) hide)
     )
@@
       (effects (font (size 1.27 1.27)) (justify left))
     )
-    (property "Footprint" "GioN_Custom:TerminalBlock_WAGO_236-412_1x12_P5.00mm_45Degree" (at 356.87 119.38 0)
+    (property "Footprint" "GioN_Custom:WAGO_250-212_1x12_P3.50mm" (at 356.87 119.38 0)
       (effects (font (size 1.27 1.27)) hide)
     )
@@
       (effects (font (size 1.27 1.27)) (justify left))
     )
-    (property "Footprint" "GioN_Custom:TerminalBlock_WAGO_236-402_1x02_P5.00mm_45Degree" (at 347.98 44.45 0)
+    (property "Footprint" "GioN_Custom:WAGO_250-202_1x02_P3.50mm" (at 347.98 44.45 0)
       (effects (font (size 1.27 1.27)) hide)
     )
@@
       (effects (font (size 1.27 1.27)) (justify left))
     )
-    (property "Footprint" "GioN_Custom:TerminalBlock_WAGO_236-402_1x02_P5.00mm_45Degree" (at 347.98 31.75 0)
+    (property "Footprint" "GioN_Custom:WAGO_250-202_1x02_P3.50mm" (at 347.98 31.75 0)
       (effects (font (size 1.27 1.27)) hide)
     )
@@
       (effects (font (size 1.27 1.27)) (justify left))
     )
-    (property "Footprint" "GioN_Custom:TerminalBlock_WAGO_236-402_1x02_P5.00mm_45Degree" (at 347.98 69.85 0)
+    (property "Footprint" "GioN_Custom:WAGO_250-202_1x02_P3.50mm" (at 347.98 69.85 0)
       (effects (font (size 1.27 1.27)) hide)
     )

Commit message: partly route pcb
Parts:
- SW10, SW11, SW12, SW13, SW9: footprint Button_Switch_SMD:SW_SPST_B3U-1000P -> GioN_Custom:SW_SPST_B3U-1000P
Changed lines of the file:
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@@
       (effects (font (size 1.27 1.27)))
     )
-    (property "Footprint" "Button_Switch_SMD:SW_SPST_B3U-1000P" (at 251.46 186.69 0)
+    (property "Footprint" "GioN_Custom:SW_SPST_B3U-1000P" (at 251.46 186.69 0)
       (effects (font (size 1.27 1.27)) hide)
     )
@@
       (effects (font (size 1.27 1.27)))
     )
-    (property "Footprint" "Button_Switch_SMD:SW_SPST_B3U-1000P" (at 219.71 217.17 0)
+    (property "Footprint" "GioN_Custom:SW_SPST_B3U-1000P" (at 219.71 217.17 0)
       (effects (font (size 1.27 1.27)) hide)
     )
@@
       (effects (font (size 1.27 1.27)))
     )
-    (property "Footprint" "Button_Switch_SMD:SW_SPST_B3U-1000P" (at 251.46 201.93 0)
+    (property "Footprint" "GioN_Custom:SW_SPST_B3U-1000P" (at 251.46 201.93 0)
       (effects (font (size 1.27 1.27)) hide)
     )
@@
       (effects (font (size 1.27 1.27)))
     )
-    (property "Footprint" "Button_Switch_SMD:SW_SPST_B3U-1000P" (at 219.71 186.69 0)
+    (property "Footprint" "GioN_Custom:SW_SPST_B3U-1000P" (at 219.71 186.69 0)
       (effects (font (size 1.27 1.27)) hide)
     )
@@
       (effects (font (size 1.27 1.27)))
     )
-    (property "Footprint" "Button_Switch_SMD:SW_SPST_B3U-1000P" (at 219.71 201.93 0)
+    (property "Footprint" "GioN_Custom:SW_SPST_B3U-1000P" (at 219.71 201.93 0)
       (effects (font (size 1.27 1.27)) hide)
     )

Commit message: Finish V2 R1
Parts:
- added D29, D30, D31, D32, D33, D34, D35, D36, D37, D38, D39: LED, LED_SMD:LED_0603_1608Metric_Pad1.05x0.95mm_HandSolder, symbol Device:LED
- added R100, R101, R102, R103, R104, R105, R106, R107, R108, R98, R99: 10k, Resistor_SMD:R_0603_1608Metric_Pad0.98x0.95mm_HandSolder, symbol Device:R
- R24: value 1k5 -> 5k6
Connections:
- net +24V: now also J10.2 (Pin_2), J11.2 (Pin_2), J12.2 (Pin_2), J13.2 (Pin_2), J14.2 (Pin_2), J15.2 (Pin_2), J16.2 (Pin_2), J16.4 (Pin_4), J16.6 (Pin_6), J16.8 (Pin_8); no longer R24.2, R33.2, R38.2, R43.2, R60.2, R61.2, R62.2, R63.2, R80.2, R81.2, R82.2
- net GND1: now also D29.1 (K), D30.1 (K), D31.1 (K), D32.1 (K), D33.1 (K), D34.1 (K), D35.1 (K), D36.1 (K), D37.1 (K), D38.1 (K), D39.1 (K); no longer J10.2 (Pin_2), J11.2 (Pin_2), J12.2 (Pin_2), J13.2 (Pin_2), J14.2 (Pin_2), J15.2 (Pin_2), J16.2 (Pin_2), J16.4 (Pin_4), J16.6 (Pin_6), J16.8 (Pin_8)
- net HOME1: now also R98.1; no longer U25.3
- net HOME2: now also R99.1; no longer U25.1
- net HOME3: now also R100.1; no longer U24.7
- net HOME4: now also R101.1; no longer U24.5
- net HOME5: now also R102.1; no longer U24.3
- net HOME6: now also R103.1; no longer U24.1
- net MACRO1: now also R104.1; no longer U25.5
- net MACRO2: now also R105.1; no longer U25.7
- net MACRO3: now also R106.1; no longer U21.1
- net PAUSE: now also R107.1; no longer U21.3
- net RESUME: now also R108.1; no longer U21.5
- new net: R61.2, U24.1
- new net: D37.2 (A), R106.2
- new net: D33.2 (A), R102.2
- new net: R33.2, U25.1
- new net: R63.2, U25.7
- new net: D32.2 (A), R101.2
- new net: D31.2 (A), R100.2
- new net: R38.2, U24.7
- new net: R82.2, U21.5
- new net: D29.2 (A), R98.2
- new net: D38.2 (A), R107.2
- new net: R81.2, U21.3
- new net: R60.2, U24.3
- new net: R24.2, U25.3
- new net: R80.2, U21.1
- new net: D39.2 (A), R108.2
- new net: D36.2 (A), R105.2
- new net: R43.2, U24.5
- new net: D35.2 (A), R104.2
- new net: R62.2, U25.5
- new net: D30.2 (A), R99.2
- new net: D34.2 (A), R103.2
Other:
- moved on the sheet: R24, R33, R38, R43, R60, R61, R62, R63, R80, R81, R82

Commit message: Add V2R1
Other:
- moved on the sheet: J10, J11, J12, J13, J14, J15, J16

Commit message: updat values
Parts:
- D29, D30, D31, D32, D33, D34, D35, D36, D37, D38, D39: value LED -> ye
Changed lines of the file:
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@@
 			)
 		)
-		(property "Value" "LED"
+		(property "Value" "ye"
 			(at 95.25 122.2374 90)
 			(effects
@@
 			)
 		)
-		(property "Value" "LED"
+		(property "Value" "ye"
 			(at 95.25 43.4974 90)
 			(effects
@@
 			)
 		)
-		(property "Value" "LED"
+		(property "Value" "ye"
 			(at 289.56 82.8674 90)
 			(effects
@@
 			)
 		)
-		(property "Value" "LED"
+		(property "Value" "ye"
 			(at 289.56 122.2374 90)
 			(effects
@@
 			)
 		)
-		(property "Value" "LED"
+		(property "Value" "ye"
 			(at 191.77 161.6074 90)
 			(effects
@@
 			)
 		)
-		(property "Value" "LED"
+		(property "Value" "ye"
 			(at 95.25 161.6074 90)
 			(effects
@@
 			)
 		)
-		(property "Value" "LED"
+		(property "Value" "ye"
 			(at 191.77 122.2374 90)
 			(effects
@@
 			)
 		)
-		(property "Value" "LED"
+		(property "Value" "ye"
 			(at 289.56 43.4974 90)
 			(effects
@@
 			)
 		)
-		(property "Value" "LED"
+		(property "Value" "ye"
 			(at 95.25 82.8674 90)
 			(effects
@@
 			)
 		)
-		(property "Value" "LED"
+		(property "Value" "ye"
 			(at 191.77 43.4974 90)
 			(effects
@@
 			)
 		)
-		(property "Value" "LED"
+		(property "Value" "ye"
 			(at 191.77 82.8674 90)
 			(effects

Commit message: Update schematic
Remove 1N4148 in PWM to 10V converter, connect test input buttons to 24V instead of ground, tune some resistors and caps
Connections:
- net +24V: now also SW10.2, SW11.2, SW12.2, SW13.2, SW9.2
- net GND1: no longer SW10.2, SW11.2, SW12.2, SW13.2, SW9.2
