File: kicad/FluidNC/outputs.kicad_sch (KiCad schematic)
At the start: 47 parts, among them J17 Conn_01x04_Socket, J20 Conn_01x04_Socket, J21 Conn_01x08_Socket, J22 Conn_01x08_Socket, J23 Conn_01x08_Socket, J24 Conn_01x08_Socket, J25 Conn_01x08_Socket, J26 Conn_01x08_Socket, J27 Conn_01x06_Pin, J3 Conn_01x03_Pin, U10 ADuM120N, U11 ADuM120N, U12 LM358, U26 ISO1H811G, U3 74HCT595, U4 74HCT595, U5 74HCT595, U6 74HCT595, U7 ISO1H811G

Commit message: USB-C CC fix
Parts:
- renumbered C5 to C13, C5 to C14, C5 to C15, C5 to C16, C5 to C17, C5 to C18, C5 to C19, C5 to C20, C5 to C21, C5 to C22, C5 to C23, C5 to C24, C5 to C72, D3 to D4, D3 to D8, J3 to J18, J3 to J19, R9 to R11, R3 to R13, R9 to R14, R3 to R15, R9 to R16, R9 to R17, R3 to R18, R9 to R19, R3 to R21, R9 to R70

Commit message: Update schematic
reduce size, changed connectors, improoved schematic
Parts:
- added D10, D9: 1N4148WS, Diode_SMD:D_SOD-323, symbol Diode:1N4148WS
- C23, C24: value 100n -> 1u
- J17, J20: footprint GioN_Custom:TerminalBlock_WAGO_236-404_1x04_P5.00mm_45Degree -> GioN_Custom:WAGO_250-204_1x04_P3.50mm
- J21, J22, J23, J24, J25, J26: footprint GioN_Custom:TerminalBlock_WAGO_236-408_1x08_P5.00mm_45Degree -> GioN_Custom:WAGO_250-208_1x08_P3.50mm
Connections:
- net PWM1: now also D9.2 (A); no longer R13.1, R14.1
- net PWM2: now also D10.2 (A); no longer R17.1, R18.1
- new net: D10.1 (K), R17.1, R18.1
- new net: D9.1 (K), R13.1, R14.1
Changed lines of the file:
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@@
     (stroke (width 0) (type default))
   )
-  (wire (pts (xy 224.79 25.4) (xy 226.06 25.4))
+  (wire (pts (xy 214.63 25.4) (xy 217.17 25.4))
     (stroke (width 0) (type default))
   )
@@
     (stroke (width 0) (type default))
   )
+  (wire (pts (xy 224.79 25.4) (xy 226.06 25.4))
+    (stroke (width 0) (type default))
+  )
   (wire (pts (xy 236.22 76.2) (xy 236.22 83.82))
     (stroke (width 0) (type default))
@@
     (stroke (width 0) (type default))
   )
-  (wire (pts (xy 224.79 60.96) (xy 226.06 60.96))
+  (wire (pts (xy 214.63 60.96) (xy 217.17 60.96))
     (stroke (width 0) (type default))
   )
@@
     (stroke (width 0) (type default))
   )
+  (wire (pts (xy 224.79 60.96) (xy 226.06 60.96))
+    (stroke (width 0) (type default))
+  )
   (wire (pts (xy 124.46 148.59) (xy 127 148.59))
     (stroke (width 0) (type default))
@@
     (stroke (width 0) (type default))
   )
-  (global_label "PWM2" (shape input) (at 224.79 60.96 180) (fields_autoplaced)
+  (global_label "PWM2" (shape input) (at 214.63 60.96 180) (fields_autoplaced)
     (effects (font (size 1.27 1.27)) (justify right))
-    (property "Intersheetrefs" "${INTERSHEET_REFS}" (at 216.4225 60.96 0)
+    (property "Intersheetrefs" "${INTERSHEET_REFS}" (at 206.2625 60.96 0)
       (effects (font (size 1.27 1.27)) (justify right) hide)
     )
@@
     )
   )
-  (global_label "PWM1" (shape input) (at 224.79 25.4 180) (fields_autoplaced)
+  (global_label "PWM1" (shape input) (at 214.63 25.4 180) (fields_autoplaced)
     (effects (font (size 1.27 1.27)) (justify right))
-    (property "Intersheetrefs" "${INTERSHEET_REFS}" (at 216.4225 25.4 0)
+    (property "Intersheetrefs" "${INTERSHEET_REFS}" (at 206.2625 25.4 0)
       (effects (font (size 1.27 1.27)) (justify right) hide)
     )
@@
       (effects (font (size 1.27 1.27)) (justify left))
     )
-    (property "Footprint" "GioN_Custom:TerminalBlock_WAGO_236-404_1x04_P5.00mm_45Degree" (at 132.08 148.59 0)
+    (property "Footprint" "GioN_Custom:WAGO_250-204_1x04_P3.50mm" (at 132.08 148.59 0)
       (effects (font (size 1.27 1.27)) hide)
     )
@@
       (effects (font (size 1.27 1.27)) (justify left))
     )
-    (property "Footprint" "GioN_Custom:TerminalBlock_WAGO_236-404_1x04_P5.00mm_45Degree" (at 133.35 180.34 0)
+    (property "Footprint" "GioN_Custom:WAGO_250-204_1x04_P3.50mm" (at 133.35 180.34 0)
       (effects (font (size 1.27 1.27)) hide)
     )
@@
     )
   )
+  (symbol (lib_id "Diode:1N4148WS") (at 220.98 60.96 180) (unit 1)
+    (in_bom yes) (on_board yes) (dnp no) (fields_autoplaced)
+    (property "Reference" "D10" (at 220.98 54.61 0)
+      (effects (font (size 1.27 1.27)))
+    )
+    (property "Value" "1N4148WS" (at 220.98 57.15 0)
+      (effects (font (size 1.27 1.27)))
+    )
+    (property "Footprint" "Diode_SMD:D_SOD-323" (at 220.98 56.515 0)
+      (effects (font (size 1.27 1.27)) hide)
+    )
+    (property "Datasheet" "https://www.vishay.com/docs/85751/1n4148ws.pdf" (at 220.98 60.96 0)
+      (effects (font (size 1.27 1.27)) hide)
+    )
+    (property "Sim.Device" "D" (at 220.98 60.96 0)
+      (effects (font (size 1.27 1.27)) hide)
+    )
+    (property "Sim.Pins" "1=K 2=A" (at 220.98 60.96 0)
+      (effects (font (size 1.27 1.27)) hide)
+    )
+    (pin "2")
+    (pin "1")
+    (instances
+      (project "FluidNC"
+        (path "/e3fd5c1c-6c47-4c53-8f48-29ce6734bbe9/19e27c1a-a8c5-4111-ac88-1c42761b7965"
+          (reference "D10") (unit 1)
+        )
+      )
+    )
+  )
   (symbol (lib_id "power:+24V") (at 128.27 172.72 0) (unit 1)
     (in_bom yes) (on_board yes) (dnp no) (fields_autoplaced)
@@
       (effects (font (size 1.27 1.27)) (justify left))
     )
-    (property "Footprint" "GioN_Custom:TerminalBlock_WAGO_236-408_1x08_P5.00mm_45Degree" (at 212.09 262.89 0)
+    (property "Footprint" "GioN_Custom:WAGO_250-208_1x08_P3.50mm" (at 212.09 262.89 0)
       (effects (font (size 1.27 1.27)) hide)
     )
@@
       (effects (font (size 1.27 1.27)))
     )
-    (property "Footprint" "GioN_Custom:TerminalBlock_WAGO_236-408_1x08_P5.00mm_45Degree" (at 185.42 243.84 0)
+    (property "Footprint" "GioN_Custom:WAGO_250-208_1x08_P3.50mm" (at 185.42 243.84 0)
       (effects (font (size 1.27 1.27)) hide)
     )
@@
       (effects (font (size 1.27 1.27)) (justify left))
     )
-    (property "Footprint" "GioN_Custom:TerminalBlock_WAGO_236-408_1x08_P5.00mm_45Degree" (at 182.88 105.41 0)
+    (property "Footprint" "GioN_Custom:WAGO_250-208_1x08_P3.50mm" (at 182.88 105.41 0)
       (effects (font (size 1.27 1.27)) hide)
     )
@@
     )
   )
+  (symbol (lib_id "Diode:1N4148WS") (at 220.98 25.4 180) (unit 1)
+    (in_bom yes) (on_board yes) (dnp no) (fields_autoplaced)
+    (property "Reference" "D9" (at 220.98 19.05 0)
+      (effects (font (size 1.27 1.27)))
+    )
+    (property "Value" "1N4148WS" (at 220.98 21.59 0)
+      (effects (font (size 1.27 1.27)))
+    )
+    (property "Footprint" "Diode_SMD:D_SOD-323" (at 220.98 20.955 0)
+      (effects (font (size 1.27 1.27)) hide)
+    )
+    (property "Datasheet" "https://www.vishay.com/docs/85751/1n4148ws.pdf" (at 220.98 25.4 0)
+      (effects (font (size 1.27 1.27)) hide)
+    )
+    (property "Sim.Device" "D" (at 220.98 25.4 0)
+      (effects (font (size 1.27 1.27)) hide)
+    )
+    (property "Sim.Pins" "1=K 2=A" (at 220.98 25.4 0)
+      (effects (font (size 1.27 1.27)) hide)
+    )
+    (pin "2")
+    (pin "1")
+    (instances
+      (project "FluidNC"
+        (path "/e3fd5c1c-6c47-4c53-8f48-29ce6734bbe9/19e27c1a-a8c5-4111-ac88-1c42761b7965"
+          (reference "D9") (unit 1)
+        )
+      )
+    )
+  )
   (symbol (lib_id "Device:R") (at 245.11 78.74 0) (unit 1)
     (in_bom yes) (on_board yes) (dnp no)
@@
       (effects (font (size 1.27 1.27)) (justify left))
     )
-    (property "Footprint" "GioN_Custom:TerminalBlock_WAGO_236-408_1x08_P5.00mm_45Degree" (at 217.17 100.33 0)
+    (property "Footprint" "GioN_Custom:WAGO_250-208_1x08_P3.50mm" (at 217.17 100.33 0)
       (effects (font (size 1.27 1.27)) hide)
     )
@@
       (effects (font (size 1.27 1.27)) (justify left))
     )
-    (property "Value" "100n" (at 240.03 73.66 0)
+    (property "Value" "1u" (at 240.03 73.66 0)
       (effects (font (size 1.27 1.27)) (justify left))
     )
@@
       (effects (font (size 1.27 1.27)) (justify left))
     )
-    (property "Value" "100n" (at 240.03 38.1 0)
+    (property "Value" "1u" (at 240.03 38.1 0)
       (effects (font (size 1.27 1.27)) (justify left))
     )
@@
       (effects (font (size 1.27 1.27)) (justify left))
     )
-    (property "Footprint" "GioN_Custom:TerminalBlock_WAGO_236-408_1x08_P5.00mm_45Degree" (at 217.17 125.73 0)
+    (property "Footprint" "GioN_Custom:WAGO_250-208_1x08_P3.50mm" (at 217.17 125.73 0)
       (effects (font (size 1.27 1.27)) hide)
     )
@@
       (effects (font (size 1.27 1.27)) (justify left))
     )
-    (property "Footprint" "GioN_Custom:TerminalBlock_WAGO_236-408_1x08_P5.00mm_45Degree" (at 217.17 149.86 0)
+    (property "Footprint" "GioN_Custom:WAGO_250-208_1x08_P3.50mm" (at 217.17 149.86 0)
       (effects (font (size 1.27 1.27)) hide)
     )

Commit message: Finish V2 R1
Parts:
- added C31, C38, C73, C74, C75, C76, C77, C78, C79, C80, C81, C82, C83, C84, C85, C86: 10n, Capacitor_SMD:C_0603_1608Metric_Pad1.08x0.95mm_HandSolder, symbol Device:C
- added D11, D12, D13, D14, D15, D16, D17, D18, D19, D20, D21, D22, D23, D24, D25, D26, D27, D28: LED, LED_SMD:LED_0603_1608Metric_Pad1.05x0.95mm_HandSolder, symbol Device:LED
- added R71, R75, R79, R83, R84, R85, R86, R87, R88, R89, R90, R91, R92, R93, R94, R95, R96, R97: 10k, Resistor_SMD:R_0603_1608Metric_Pad0.98x0.95mm_HandSolder, symbol Device:R
Connections:
- net GND1: now also C31.2, C38.2, C73.2, C74.2, C75.2, C76.2, C77.2, C78.2, C79.2, C80.2, C81.2, C82.2, C83.2, C84.2, C85.2, C86.2, D27.1 (K), D28.1 (K), R71.2, R75.2, R79.2, R83.2, R84.2, R85.2, R86.2, R87.2, R88.2, R89.2, R90.2, R91.2, R92.2, R93.2, R94.2, R95.2
- net PWM1: now also R96.1
- net PWM2: now also R97.1
- net at J25.1 (Pin_1), U26.21 (OUT7), U26.22 (OUT7): now also C86.1, D26.2 (A)
- net at J25.2 (Pin_2), U26.23 (OUT6), U26.24 (OUT6): now also C85.1, D25.2 (A)
- net at J25.3 (Pin_3), U26.25 (OUT5), U26.26 (OUT5): now also C84.1, D24.2 (A)
- net at J25.4 (Pin_4), U26.27 (OUT4), U26.28 (OUT4): now also C83.1, D23.2 (A)
- net at J25.5 (Pin_5), U26.29 (OUT3), U26.30 (OUT3): now also C82.1, D22.2 (A)
- net at J25.6 (Pin_6), U26.31 (OUT2), U26.32 (OUT2): now also C81.1, D21.2 (A)
- net at J25.7 (Pin_7), U26.33 (OUT1), U26.34 (OUT1): now also C80.1, D20.2 (A)
- net at J25.8 (Pin_8), U26.35 (OUT0), U26.36 (OUT0): now also C79.1, D19.2 (A)
- net at J21.1 (Pin_1), U7.21 (OUT7), U7.22 (OUT7): now also C78.1, D18.2 (A)
- net at J21.2 (Pin_2), U7.23 (OUT6), U7.24 (OUT6): now also C77.1, D17.2 (A)
- net at J21.3 (Pin_3), U7.25 (OUT5), U7.26 (OUT5): now also C76.1, D16.2 (A)
- net at J21.4 (Pin_4), U7.27 (OUT4), U7.28 (OUT4): now also C75.1, D15.2 (A)
- net at J21.5 (Pin_5), U7.29 (OUT3), U7.30 (OUT3): now also C74.1, D14.2 (A)
- net at J21.6 (Pin_6), U7.31 (OUT2), U7.32 (OUT2): now also C73.1, D13.2 (A)
- net at J21.7 (Pin_7), U7.33 (OUT1), U7.34 (OUT1): now also C38.1, D12.2 (A)
- net at J21.8 (Pin_8), U7.35 (OUT0), U7.36 (OUT0): now also C31.1, D11.2 (A)
- new net: D19.1 (K), R88.1
- new net: D12.1 (K), R75.1
- new net: D18.1 (K), R87.1
- new net: D14.1 (K), R83.1
- new net: D23.1 (K), R92.1
- new net: D16.1 (K), R85.1
- new net: D20.1 (K), R89.1
- new net: D22.1 (K), R91.1
- new net: D28.2 (A), R97.2
- new net: D27.2 (A), R96.2
- new net: D17.1 (K), R86.1
- new net: D11.1 (K), R71.1
- new net: D21.1 (K), R90.1
- new net: D15.1 (K), R84.1
- new net: D24.1 (K), R93.1
- new net: D25.1 (K), R94.1
- new net: D13.1 (K), R79.1
- new net: D26.1 (K), R95.1
Other:
- moved on the sheet: C22, C72, D8, J21, J22, J23, J24, J25, J26, R70, U12C, U26

Commit message: Add debug features
Change PCB Color
Add ground pins for probing
Add debug leds for step, dir and stepper_en
Add silkscreen with pin definitions
Parts:
- added D40, D41, D42, D43, D44, D45, D46, D47, D48, D49, D50, D51, D52: LED, LED_SMD:LED_0603_1608Metric_Pad1.05x0.95mm_HandSolder, symbol Device:LED
- added J2, J28, J29, J3, J30, J32: Conn_01x01_Pin, Connector_PinHeader_2.54mm:PinHeader_1x01_P2.54mm_Vertical, symbol Connector:Conn_01x01_Pin
- added R109, R110, R111, R112, R113, R114, R115, R116, R117, R118, R119, R120, R121: 10k, Resistor_SMD:R_0603_1608Metric_Pad0.98x0.95mm_HandSolder, symbol Device:R
Connections:
- net GND: now also D40.1 (K), D41.1 (K), D42.1 (K), D43.1 (K), D44.1 (K), D45.1 (K), D46.1 (K), D47.1 (K), D48.1 (K), D49.1 (K), D50.1 (K), D51.1 (K), D52.1 (K), J2.1 (Pin_1), J28.1 (Pin_1), J3.1 (Pin_1)
- net GND1: now also J29.1 (Pin_1), J30.1 (Pin_1), J32.1 (Pin_1)
- net I2SO0_DIR6: now also R109.1
- net I2SO10_DIR1: now also R119.1
- net I2SO11_STEP1: now also R120.1
- net I2SO14_EN_STEPPER: now also R121.1
- net I2SO1_STEP6: now also R110.1
- net I2SO2_DIR5: now also R111.1
- net I2SO3_STEP5: now also R112.1
- net I2SO4_DIR4: now also R113.1
- net I2SO5_STEP4: now also R114.1
- net I2SO6_DIR3: now also R115.1
- net I2SO7_STEP3: now also R116.1
- net I2SO8_DIR2: now also R117.1
- net I2SO9_STEP2: now also R118.1
- new net: D47.2 (A), R116.2
- new net: D52.2 (A), R121.2
- new net: D45.2 (A), R114.2
- new net: D43.2 (A), R112.2
- new net: D49.2 (A), R118.2
- new net: D42.2 (A), R111.2
- new net: D40.2 (A), R109.2
- new net: D48.2 (A), R117.2
- new net: D44.2 (A), R113.2
- new net: D46.2 (A), R115.2
- new net: D51.2 (A), R120.2
- new net: D41.2 (A), R110.2
- new net: D50.2 (A), R119.2

Commit message: Add V2R1
Other:
- moved on the sheet: C22, C72, C79, C80, C81, C82, C83, C84, C85, C86, D19, D20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

Commit message: updat values
Parts:
- D11, D12, D13, D14, D15, D16, D17, D18, D19, D20, D21, D22, D23, D24, D25, D26, D27, D28, D4, D40, D41, D42, D43, D44, D45, D46, D47, D48, D49, D50, D51, D52, D8: value LED -> rt
Changed lines of the file:
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@@
 			)
 		)
-		(property "Value" "LED"
+		(property "Value" "rt"
 			(at 181.61 195.8974 90)
 			(effects
@@
 			)
 		)
-		(property "Value" "LED"
+		(property "Value" "rt"
 			(at 133.35 149.86 90)
 			(effects
@@
 			)
 		)
-		(property "Value" "LED"
+		(property "Value" "rt"
 			(at 306.07 126.0474 90)
 			(effects
@@
 			)
 		)
-		(property "Value" "LED"
+		(property "Value" "rt"
 			(at 234.95 126.0474 90)
 			(effects
@@
 			)
 		)
-		(property "Value" "LED"
+		(property "Value" "rt"
 			(at 199.39 126.0474 90)
 			(effects
@@
 			)
 		)
-		(property "Value" "LED"
+		(property "Value" "rt"
 			(at 252.73 195.8974 90)
 			(effects
@@
 			)
 		)
-		(property "Value" "LED"
+		(property "Value" "rt"
 			(at 52.07 274.6374 90)
 			(effects
@@
 			)
 		)
-		(property "Value" "LED"
+		(property "Value" "rt"
 			(at 41.91 274.6374 90)
 			(effects
@@
 			)
 		)
-		(property "Value" "LED"
+		(property "Value" "rt"
 			(at 102.87 274.6374 90)
 			(effects
@@
 			)
 		)
-		(property "Value" "LED"
+		(property "Value" "rt"
 			(at 21.59 274.6374 90)
 			(effects
@@
 			)
 		)
-		(property "Value" "LED"
+		(property "Value" "rt"
 			(at 215.9 42.2274 90)
 			(effects
@@
 			)
 		)
-		(property "Value" "LED"
+		(property "Value" "rt"
 			(at 217.17 77.7874 90)
 			(effects
@@
 			)
 		)
-		(property "Value" "LED"
+		(property "Value" "rt"
 			(at 288.29 126.0474 90)
 			(effects
@@
 			)
 		)
-		(property "Value" "LED"
+		(property "Value" "rt"
 			(at 234.95 195.8974 90)
 			(effects
@@
 			)
 		)
-		(property "Value" "LED"
+		(property "Value" "rt"
 			(at 181.61 126.0474 90)
 			(effects
@@
 			)
 		)
-		(property "Value" "LED"
+		(property "Value" "rt"
 			(at 270.51 126.0474 90)
 			(effects
@@
 			)
 		)
-		(property "Value" "LED"
+		(property "Value" "rt"
 			(at 92.71 274.6374 90)
 			(effects
@@
 			)
 		)
-		(property "Value" "LED"
+		(property "Value" "rt"
 			(at 133.35 77.47 90)
 			(effects
@@
 			)
 		)
-		(property "Value" "LED"
+		(property "Value" "rt"
 			(at 72.39 274.6374 90)
 			(effects
@@
 			)
 		)
-		(property "Value" "LED"
+		(property "Value" "rt"
 			(at 82.55 274.6374 90)
 			(effects
@@
 			)
 		)
-		(property "Value" "LED"
+		(property "Value" "rt"
 			(at 252.73 126.0474 90)
 			(effects
@@
 			)
 		)
-		(property "Value" "LED"
+		(property "Value" "rt"
 			(at 270.51 195.8974 90)
 			(effects
@@
 			)
 		)
-		(property "Value" "LED"
+		(property "Value" "rt"
 			(at 288.29 195.8974 90)
 			(effects
@@
 			)
 		)
-		(property "Value" "LED"
+		(property "Value" "rt"
 			(at 143.51 274.6374 90)
 			(effects
@@
 			)
 		)
-		(property "Value" "LED"
+		(property "Value" "rt"
 			(at 62.23 274.6374 90)
 			(effects
@@
 			)
 		)
-		(property "Value" "LED"
+		(property "Value" "rt"
 			(at 31.75 274.6374 90)
 			(effects
@@
 			)
 		)
-		(property "Value" "LED"
+		(property "Value" "rt"
 			(at 217.17 195.8974 90)
 			(effects
@@
 			)
 		)
-		(property "Value" "LED"
+		(property "Value" "rt"
 			(at 133.35 274.6374 90)
 			(effects
@@
 			)
 		)
-		(property "Value" "LED"
+		(property "Value" "rt"
 			(at 217.17 126.0474 90)
 			(effects
@@
 			)
 		)
-		(property "Value" "LED"
+		(property "Value" "rt"
 			(at 123.19 274.6374 90)
 			(effects
@@
 			)
 		)
-		(property "Value" "LED"
+		(property "Value" "rt"
 			(at 113.03 274.6374 90)
 			(effects
@@
 			)
 		)
-		(property "Value" "LED"
+		(property "Value" "rt"
 			(at 306.07 195.8974 90)
 			(effects
@@
 			)
 		)
-		(property "Value" "LED"
+		(property "Value" "rt"
 			(at 199.39 195.8974 90)
 			(effects

Commit message: Update schematic
Remove 1N4148 in PWM to 10V converter, connect test input buttons to 24V instead of ground, tune some resistors and caps
Parts:
- removed D10, D9: 1N4148WS, Diode_SMD:D_SOD-323, symbol Diode:1N4148WS
- C23, C24: value 1u -> 100n
- R13, R18: value 100R -> 10k
- R96, R97: value 10k -> 5k1
Connections:
- net PWM1: now also R13.1, R14.1
- net PWM2: now also R17.1, R18.1
Changed lines of the file:
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@@
 	(wire
 		(pts
-			(xy 212.09 25.4) (xy 217.17 25.4)
+			(xy 212.09 25.4) (xy 226.06 25.4)
 		)
 		(stroke
@@
 	(wire
 		(pts
-			(xy 224.79 25.4) (xy 226.06 25.4)
-		)
-		(stroke
-			(width 0)
-			(type default)
-		)
-	)
-	(wire
-		(pts
 			(xy 240.03 137.16) (xy 248.92 137.16)
 		)
@@
 	(wire
 		(pts
-			(xy 224.79 60.96) (xy 226.06 60.96)
-		)
-		(stroke
-			(width 0)
-			(type default)
-		)
-	)
-	(wire
-		(pts
 			(xy 266.7 187.96) (xy 266.7 189.23)
 		)
@@
 	(wire
 		(pts
-			(xy 213.36 60.96) (xy 217.17 60.96)
+			(xy 213.36 60.96) (xy 226.06 60.96)
 		)
 		(stroke
@@
 	)
 	(symbol
-		(lib_id "Diode:1N4148WS")
-		(at 220.98 60.96 180)
-		(unit 1)
-		(exclude_from_sim no)
-		(in_bom yes)
-		(on_board yes)
-		(dnp no)
-		(fields_autoplaced yes)
-		(property "Reference" "D10"
-			(at 220.98 54.61 0)
-			(effects
-				(font
-					(size 1.27 1.27)
-				)
-			)
-		)
-		(property "Value" "1N4148WS"
-			(at 220.98 57.15 0)
-			(effects
-				(font
-					(size 1.27 1.27)
-				)
-			)
-		)
-		(property "Footprint" "Diode_SMD:D_SOD-323"
-			(at 220.98 56.515 0)
-			(effects
-				(font
-					(size 1.27 1.27)
-				)
-				(hide yes)
-			)
-		)
-		(property "Datasheet" "https://www.vishay.com/docs/85751/1n4148ws.pdf"
-			(at 220.98 60.96 0)
-			(effects
-				(font
-					(size 1.27 1.27)
-				)
-				(hide yes)
-			)
-		)
-		(property "Description" ""
-			(at 220.98 60.96 0)
-			(effects
-				(font
-					(size 1.27 1.27)
-				)
-				(hide yes)
-			)
-		)
-		(property "Sim.Device" "D"
-			(at 220.98 60.96 0)
-			(effects
-				(font
-					(size 1.27 1.27)
-				)
-				(hide yes)
-			)
-		)
-		(property "Sim.Pins" "1=K 2=A"
-			(at 220.98 60.96 0)
-			(effects
-				(font
-					(size 1.27 1.27)
-				)
-				(hide yes)
-			)
-		)
-		(pin "2"
-		)
-		(pin "1"
-		)
-		(instances
-			(project "FluidNC"
-				(path "/e3fd5c1c-6c47-4c53-8f48-29ce6734bbe9/19e27c1a-a8c5-4111-ac88-1c42761b7965"
-					(reference "D10")
-					(unit 1)
-				)
-			)
-		)
-	)
-	(symbol
 		(lib_id "Device:R")
 		(at 109.22 262.89 0)
@@
 			)
 		)
-		(property "Value" "100R"
+		(property "Value" "10k"
 			(at 231.14 22.86 90)
 			(effects
@@
 			)
 		)
-		(property "Value" "10k"
+		(property "Value" "5k1"
 			(at 215.9 67.31 0)
 			(effects
@@
 			)
 		)
-		(property "Value" "10k"
+		(property "Value" "5k1"
 			(at 214.63 31.75 0)
 			(effects
@@
 	)
 	(symbol
-		(lib_id "Diode:1N4148WS")
-		(at 220.98 25.4 180)
-		(unit 1)
-		(exclude_from_sim no)
-		(in_bom yes)
-		(on_board yes)
-		(dnp no)
-		(fields_autoplaced yes)
-		(property "Reference" "D9"
-			(at 220.98 19.05 0)
-			(effects
-				(font
-					(size 1.27 1.27)
-				)
-			)
-		)
-		(property "Value" "1N4148WS"
-			(at 220.98 21.59 0)
-			(effects
-				(font
-					(size 1.27 1.27)
-				)
-			)
-		)
-		(property "Footprint" "Diode_SMD:D_SOD-323"
-			(at 220.98 20.955 0)
-			(effects
-				(font
-					(size 1.27 1.27)
-				)
-				(hide yes)
-			)
-		)
-		(property "Datasheet" "https://www.vishay.com/docs/85751/1n4148ws.pdf"
-			(at 220.98 25.4 0)
-			(effects
-				(font
-					(size 1.27 1.27)
-				)
-				(hide yes)
-			)
-		)
-		(property "Description" ""
-			(at 220.98 25.4 0)
-			(effects
-				(font
-					(size 1.27 1.27)
-				)
-				(hide yes)
-			)
-		)
-		(property "Sim.Device" "D"
-			(at 220.98 25.4 0)
-			(effects
-				(font
-					(size 1.27 1.27)
-				)
-				(hide yes)
-			)
-		)
-		(property "Sim.Pins" "1=K 2=A"
-			(at 220.98 25.4 0)
-			(effects
-				(font
-					(size 1.27 1.27)
-				)
-				(hide yes)
-			)
-		)
-		(pin "2"
-		)
-		(pin "1"
-		)
-		(instances
-			(project "FluidNC"
-				(path "/e3fd5c1c-6c47-4c53-8f48-29ce6734bbe9/19e27c1a-a8c5-4111-ac88-1c42761b7965"
-					(reference "D9")
-					(unit 1)
-				)
-			)
-		)
-	)
-	(symbol
 		(lib_id "Device:R")
 		(at 213.36 201.93 0)
@@
 		(fields_autoplaced yes)
 		(property "Reference" "C24"
-			(at 240.03 71.12 0)
+			(at 240.03 71.1199 0)
 			(effects
 				(font
@@
 			)
 		)
-		(property "Value" "1u"
-			(at 240.03 73.66 0)
+		(property "Value" "100n"
+			(at 240.03 73.6599 0)
 			(effects
 				(font
@@
 			)
 		)
-		(property "Value" "100R"
+		(property "Value" "10k"
 			(at 231.14 58.42 90)
 			(effects
@@
 		(fields_autoplaced yes)
 		(property "Reference" "C23"
-			(at 240.03 35.56 0)
+			(at 240.03 35.5599 0)
 			(effects
 				(font
@@
 			)
 		)
-		(property "Value" "1u"
-			(at 240.03 38.1 0)
+		(property "Value" "100n"
+			(at 240.03 38.0999 0)
 			(effects
 				(font
