File: kicad/FluidNC/FluidNC.kicad_sch (KiCad schematic)
At the start: 45 parts, among them J1 USB_C_Receptacle_USB2.0, J15 Conn_01x02_Socket, Q1 BC847, Q2 BC847, SW1 SW_RESET, SW2 SW_BOOT, U1 CH340C, U2 ESP32-WROOM-32, U8 NCP1117-3.3_SOT223, U9 LM2596S-5

Commit message: USB-C CC fix
Parts:
- renumbered J15 to J31
Connections:
- net at J1.A5 (CC1): now also R1.1
- net at J1.A8 (SBU1): no longer R2.1
- net at J1.B5 (CC2): now also R2.1
- net at J1.B8 (SBU2): no longer R1.1
Other:
- moved on the sheet: R1, R2
Changed lines of the file:
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@@
 (kicad_sch (version 20230121) (generator eeschema)
   (paper "A4")
+  (junction (at 53.34 63.5) (diameter 0) (color 0 0 0 0)
+  )
   (junction (at 148.59 78.74) (diameter 0) (color 0 0 0 0)
   )
@@
   (junction (at 177.8 142.24) (diameter 0) (color 0 0 0 0)
   )
-  (junction (at 43.18 63.5) (diameter 0) (color 0 0 0 0)
-  )
   (junction (at 242.57 39.37) (diameter 0) (color 0 0 0 0)
   )
@@
     (stroke (width 0) (type default))
   )
+  (wire (pts (xy 53.34 63.5) (xy 59.69 63.5))
+    (stroke (width 0) (type default))
+  )
   (wire (pts (xy 121.92 102.87) (xy 121.92 91.44))
     (stroke (width 0) (type default))
@@
     (stroke (width 0) (type default))
   )
-  (wire (pts (xy 50.8 63.5) (xy 50.8 60.96))
+  (wire (pts (xy 53.34 63.5) (xy 53.34 60.96))
     (stroke (width 0) (type default))
   )
@@
     (stroke (width 0) (type default))
   )
-  (wire (pts (xy 43.18 52.07) (xy 43.18 53.34))
+  (wire (pts (xy 59.69 26.67) (xy 59.69 53.34))
     (stroke (width 0) (type default))
   )
@@
     (stroke (width 0) (type default))
   )
+  (wire (pts (xy 41.91 29.21) (xy 53.34 29.21))
+    (stroke (width 0) (type default))
+  )
   (wire (pts (xy 99.06 102.87) (xy 100.33 102.87))
     (stroke (width 0) (type default))
@@
     (stroke (width 0) (type default))
   )
-  (wire (pts (xy 41.91 52.07) (xy 43.18 52.07))
-    (stroke (width 0) (type default))
-  )
   (wire (pts (xy 215.9 36.83) (xy 215.9 39.37))
     (stroke (width 0) (type default))
@@
     (stroke (width 0) (type default))
   )
-  (wire (pts (xy 43.18 63.5) (xy 50.8 63.5))
-    (stroke (width 0) (type default))
-  )
-  (wire (pts (xy 50.8 49.53) (xy 50.8 53.34))
+  (wire (pts (xy 53.34 29.21) (xy 53.34 53.34))
     (stroke (width 0) (type default))
   )
@@
     (stroke (width 0) (type default))
   )
-  (wire (pts (xy 41.91 49.53) (xy 50.8 49.53))
-    (stroke (width 0) (type default))
-  )
   (wire (pts (xy 99.06 24.13) (xy 99.06 21.59))
     (stroke (width 0) (type default))
@@
     (stroke (width 0) (type default))
   )
-  (wire (pts (xy 43.18 60.96) (xy 43.18 63.5))
+  (wire (pts (xy 59.69 60.96) (xy 59.69 63.5))
     (stroke (width 0) (type default))
   )
@@
     (stroke (width 0) (type default))
   )
+  (wire (pts (xy 26.67 63.5) (xy 53.34 63.5))
+    (stroke (width 0) (type default))
+  )
   (wire (pts (xy 213.36 128.27) (xy 238.76 128.27))
     (stroke (width 0) (type default))
@@
     (stroke (width 0) (type default))
   )
-  (wire (pts (xy 26.67 63.5) (xy 43.18 63.5))
-    (stroke (width 0) (type default))
-  )
   (wire (pts (xy 172.72 39.37) (xy 149.86 39.37))
     (stroke (width 0) (type default))
@@
   )
   (wire (pts (xy 165.1 129.54) (xy 165.1 128.27))
+    (stroke (width 0) (type default))
+  )
+  (wire (pts (xy 59.69 26.67) (xy 41.91 26.67))
     (stroke (width 0) (type default))
   )
@@
   (symbol (lib_id "Connector:Conn_01x02_Socket") (at 134.62 128.27 0) (mirror y) (unit 1)
     (in_bom yes) (on_board yes) (dnp no)
-    (property "Reference" "J15" (at 133.35 128.27 0)
+    (property "Reference" "J31" (at 133.35 128.27 0)
       (effects (font (size 1.27 1.27)) (justify left))
     )
@@
     (instances
       (project "FluidNC"
-        (path "/e3fd5c1c-6c47-4c53-8f48-29ce6734bbe9/2c48d8bb-28b3-408f-91d3-bb9a92045867"
-          (reference "J15") (unit 1)
-        )
         (path "/e3fd5c1c-6c47-4c53-8f48-29ce6734bbe9"
           (reference "J31") (unit 1)
@@
     )
   )
-  (symbol (lib_id "Device:R") (at 50.8 57.15 0) (unit 1)
-    (in_bom yes) (on_board yes) (dnp no)
-    (property "Reference" "R2" (at 52.07 55.88 0)
-      (effects (font (size 1.27 1.27)) (justify left))
-    )
-    (property "Value" "5k1" (at 52.07 58.42 0)
-      (effects (font (size 1.27 1.27)) (justify left))
-    )
-    (property "Footprint" "Resistor_SMD:R_0603_1608Metric_Pad0.98x0.95mm_HandSolder" (at 49.022 57.15 90)
-      (effects (font (size 1.27 1.27)) hide)
-    )
-    (property "Datasheet" "~" (at 50.8 57.15 0)
+  (symbol (lib_id "Device:R") (at 53.34 57.15 0) (unit 1)
+    (in_bom yes) (on_board yes) (dnp no)
+    (property "Reference" "R2" (at 54.61 55.88 0)
+      (effects (font (size 1.27 1.27)) (justify left))
+    )
+    (property "Value" "5k1" (at 54.61 58.42 0)
+      (effects (font (size 1.27 1.27)) (justify left))
+    )
+    (property "Footprint" "Resistor_SMD:R_0603_1608Metric_Pad0.98x0.95mm_HandSolder" (at 51.562 57.15 90)
+      (effects (font (size 1.27 1.27)) hide)
+    )
+    (property "Datasheet" "~" (at 53.34 57.15 0)
       (effects (font (size 1.27 1.27)) hide)
     )
@@
     )
   )
-  (symbol (lib_id "Device:R") (at 43.18 57.15 0) (unit 1)
-    (in_bom yes) (on_board yes) (dnp no)
-    (property "Reference" "R1" (at 44.45 55.88 0)
-      (effects (font (size 1.27 1.27)) (justify left))
-    )
-    (property "Value" "5k1" (at 44.45 58.42 0)
-      (effects (font (size 1.27 1.27)) (justify left))
-    )
-    (property "Footprint" "Resistor_SMD:R_0603_1608Metric_Pad0.98x0.95mm_HandSolder" (at 41.402 57.15 90)
-      (effects (font (size 1.27 1.27)) hide)
-    )
-    (property "Datasheet" "~" (at 43.18 57.15 0)
-      (effects (font (size 1.27 1.27)) hide)
-    )
+  (symbol (lib_id "Device:R") (at 59.69 57.15 0) (unit 1)
+    (in_bom yes) (on_board yes) (dnp no)
+    (property "Reference" "R1" (at 60.96 55.88 0)
+      (effects (font (size 1.27 1.27)) (justify left))
+    )
+    (property "Value" "5k1" (at 60.96 58.42 0)
+      (effects (font (size 1.27 1.27)) (justify left))
+    )
+    (property "Footprint" "Resistor_SMD:R_0603_1608Metric_Pad0.98x0.95mm_HandSolder" (at 57.912 57.15 90)
+      (effects (font (size 1.27 1.27)) hide)
+    )
+    (property "Datasheet" "~" (at 59.69 57.15 0)
+      (effects (font (size 1.27 1.27)) hide)
+    )

Commit message: Update schematic
reduce size, changed connectors, improoved schematic
Parts:
- J31: footprint GioN_Custom:TerminalBlock_WAGO_236-402_1x02_P5.00mm_45Degree -> GioN_Custom:WAGO_250-202_1x02_P3.50mm
- L1: footprint Inductor_SMD:L_Changjiang_FNR5020S -> Inductor_SMD:L_7.3x7.3_H3.5
Changed lines of the file:
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@@
       (effects (font (size 1.27 1.27)) (justify left))
     )
-    (property "Footprint" "GioN_Custom:TerminalBlock_WAGO_236-402_1x02_P5.00mm_45Degree" (at 134.62 128.27 0)
+    (property "Footprint" "GioN_Custom:WAGO_250-202_1x02_P3.50mm" (at 134.62 128.27 0)
       (effects (font (size 1.27 1.27)) hide)
     )
@@
       (effects (font (size 1.27 1.27)))
     )
-    (property "Footprint" "Inductor_SMD:L_Changjiang_FNR5020S" (at 224.79 133.35 0)
-      (effects (font (size 1.27 1.27)) hide)
-    )
+    (property "Footprint" "Inductor_SMD:L_7.3x7.3_H3.5" (at 224.79 133.35 0)
+      (effects (font (size 1.27 1.27)) hide)
+    )

Commit message: partly route pcb
Parts:
- SW1, SW2: footprint Button_Switch_SMD:SW_SPST_B3U-1000P -> GioN_Custom:SW_SPST_B3U-1000P
Changed lines of the file:
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@@
       (effects (font (size 1.27 1.27)))
     )
-    (property "Footprint" "Button_Switch_SMD:SW_SPST_B3U-1000P" (at 157.48 66.04 0)
+    (property "Footprint" "GioN_Custom:SW_SPST_B3U-1000P" (at 157.48 66.04 0)
       (effects (font (size 1.27 1.27)) hide)
     )
@@
       (effects (font (size 1.27 1.27)))
     )
-    (property "Footprint" "Button_Switch_SMD:SW_SPST_B3U-1000P" (at 157.48 88.9 0)
+    (property "Footprint" "GioN_Custom:SW_SPST_B3U-1000P" (at 157.48 88.9 0)
       (effects (font (size 1.27 1.27)) hide)
     )

Commit message: Add V2R1
Other:
- removed sheet Debug
- moved on the sheet: C11, C2, C3, C39, C4, C40, C41, C9, D6, F1, J31, R1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

Commit message: updat values
Parts:
- D2, D3: value LED -> bl
- D6, D7: value LED -> gn
Changed lines of the file:
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@@
 			)
 		)
-		(property "Value" "LED"
+		(property "Value" "gn"
 			(at 271.78 24.13 0)
 			(effects
@@
 			)
 		)
-		(property "Value" "LED"
+		(property "Value" "gn"
 			(at 256.54 123.19 0)
 			(effects
@@
 			)
 		)
-		(property "Value" "LED"
+		(property "Value" "bl"
 			(at 114.3 100.33 0)
 			(effects
@@
 			)
 		)
-		(property "Value" "LED"
+		(property "Value" "bl"
 			(at 114.3 88.9 0)
 			(effects

Commit message: Minor changes
Add designated 3.2mm hole footprints,
update packages
Parts:
- D1: footprint Diode_SMD:D_SOD-323 -> Diode_SMD:D_SOD-323_HandSoldering
- D5: value D_Schottky -> SS34; footprint Diode_SMD:D_SMC -> Diode_SMD:D_SMA
- L1: footprint Inductor_SMD:L_7.3x7.3_H3.5 -> Inductor_SMD:L_6.3x6.3_H3
Changed lines of the file:
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@@
 			)
 		)
-		(property "Footprint" "Diode_SMD:D_SOD-323"
+		(property "Footprint" "Diode_SMD:D_SOD-323_HandSoldering"
 			(at 48.26 17.145 0)
 			(effects
@@
 			)
 		)
-		(property "Footprint" "Inductor_SMD:L_7.3x7.3_H3.5"
+		(property "Footprint" "Inductor_SMD:L_6.3x6.3_H3"
 			(at 224.79 133.35 0)
 			(effects
@@
 		(fields_autoplaced yes)
 		(property "Reference" "D5"
-			(at 220.98 138.1125 90)
-			(effects
-				(font
-					(size 1.27 1.27)
-				)
-				(justify left)
-			)
-		)
-		(property "Value" "D_Schottky"
-			(at 220.98 140.6525 90)
-			(effects
-				(font
-					(size 1.27 1.27)
-				)
-				(justify left)
-			)
-		)
-		(property "Footprint" "Diode_SMD:D_SMC"
+			(at 220.98 138.1124 90)
+			(effects
+				(font
+					(size 1.27 1.27)
+				)
+				(justify left)
+			)
+		)
+		(property "Value" "SS34"
+			(at 220.98 140.6524 90)
+			(effects
+				(font
+					(size 1.27 1.27)
+				)
+				(justify left)
+			)
+		)
+		(property "Footprint" "Diode_SMD:D_SMA"
 			(at 218.44 139.7 0)
 			(effects
