File: kicad/FluidNC/stepperDriver.kicad_sch (KiCad schematic)
At the start: 48 parts, among them J2 Conn_01x03_Pin, J3 Conn_01x03_Pin, J4 Conn_01x05_Socket, J5 Conn_01x05_Socket, J6 Conn_01x05_Socket, J7 Conn_01x05_Socket, J8 Conn_01x05_Socket, J9 Conn_01x05_Socket, SW3 SW_DIP_x03, SW4 SW_DIP_x03, SW5 SW_DIP_x03, SW6 SW_DIP_x03, SW7 SW_DIP_x03, SW8 SW_DIP_x03, U10 ADuM120N, U14 ULN2003A, U20 ULN2003A

Commit message: USB-C CC fix
Parts:
- renumbered C5 to C25, C5 to C26, C5 to C27, C5 to C28, C5 to C29, C5 to C30, C5 to C31, C5 to C32, C5 to C33, C5 to C34, C5 to C35, C5 to C36, C5 to C37, C5 to C38, C9 to C42, C9 to C43, C9 to C44, C9 to C45, C9 to C46, C9 to C47, U10 to U13, U10 to U15, U10 to U16, U10 to U17, U10 to U18, U10 to U19

Commit message: remove uln2003
Parts:
- removed C31, C38: 100n, Capacitor_SMD:C_0603_1608Metric_Pad1.08x0.95mm_HandSolder, symbol Device:C
- removed J2, J3: Conn_01x03_Pin, Connector_PinHeader_2.54mm:PinHeader_1x03_P2.54mm_Vertical, symbol Connector:Conn_01x03_Pin
- removed U14, U20: ULN2003A, Package_SO:SO-16_3.9x9.9mm_P1.27mm, symbol Transistor_Array:ULN2003A
Connections:
- net DIR1: now also U13.6 (VOB)
- net DIR2: now also U15.6 (VOB)
- net DIR3: now also U16.6 (VOB)
- net DIR4: now also U17.6 (VOB)
- net DIR5: now also U18.6 (VOB)
- net DIR6: now also U19.6 (VOB)
- net STEP1: now also U13.7 (VOA)
- net STEP2: now also U15.7 (VOA)
- net STEP3: now also U16.7 (VOA)
- net STEP4: now also U17.7 (VOA)
- net STEP5: now also U18.7 (VOA)
- net STEP6: now also U19.7 (VOA)

Commit message: Update schematic
reduce size, changed connectors, improoved schematic
Parts:
- J4, J5, J6, J7, J8, J9: footprint GioN_Custom:TerminalBlock_WAGO_236-405_1x05_P5.00mm_45Degree -> GioN_Custom:WAGO_250-205_1x05_P3.50mm
Changed lines of the file:
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@@
       (effects (font (size 1.27 1.27)) (justify left))
     )
-    (property "Footprint" "GioN_Custom:TerminalBlock_WAGO_236-405_1x05_P5.00mm_45Degree" (at 273.05 38.1 0)
+    (property "Footprint" "GioN_Custom:WAGO_250-205_1x05_P3.50mm" (at 273.05 38.1 0)
       (effects (font (size 1.27 1.27)) hide)
     )
@@
       (effects (font (size 1.27 1.27)) (justify left))
     )
-    (property "Footprint" "GioN_Custom:TerminalBlock_WAGO_236-405_1x05_P5.00mm_45Degree" (at 382.27 144.78 0)
+    (property "Footprint" "GioN_Custom:WAGO_250-205_1x05_P3.50mm" (at 382.27 144.78 0)
       (effects (font (size 1.27 1.27)) hide)
     )
@@
       (effects (font (size 1.27 1.27)) (justify left))
     )
-    (property "Footprint" "GioN_Custom:TerminalBlock_WAGO_236-405_1x05_P5.00mm_45Degree" (at 273.05 144.78 0)
+    (property "Footprint" "GioN_Custom:WAGO_250-205_1x05_P3.50mm" (at 273.05 144.78 0)
       (effects (font (size 1.27 1.27)) hide)
     )
@@
       (effects (font (size 1.27 1.27)) (justify left))
     )
-    (property "Footprint" "GioN_Custom:TerminalBlock_WAGO_236-405_1x05_P5.00mm_45Degree" (at 382.27 91.44 0)
+    (property "Footprint" "GioN_Custom:WAGO_250-205_1x05_P3.50mm" (at 382.27 91.44 0)
       (effects (font (size 1.27 1.27)) hide)
     )
@@
       (effects (font (size 1.27 1.27)) (justify left))
     )
-    (property "Footprint" "GioN_Custom:TerminalBlock_WAGO_236-405_1x05_P5.00mm_45Degree" (at 273.05 91.44 0)
+    (property "Footprint" "GioN_Custom:WAGO_250-205_1x05_P3.50mm" (at 273.05 91.44 0)
       (effects (font (size 1.27 1.27)) hide)
     )
@@
       (effects (font (size 1.27 1.27)) (justify left))
     )
-    (property "Footprint" "GioN_Custom:TerminalBlock_WAGO_236-405_1x05_P5.00mm_45Degree" (at 382.27 38.1 0)
-      (effects (font (size 1.27 1.27)) hide)
-    )
+    (property "Footprint" "GioN_Custom:WAGO_250-205_1x05_P3.50mm" (at 382.27 38.1 0)
+      (effects (font (size 1.27 1.27)) hide)
+    )

Commit message: Minor changes
Add designated 3.2mm hole footprints,
update packages
Parts:
- C42, C43, C44, C45, C46, C47: footprint Capacitor_SMD:CP_Elec_10x7.9 -> Capacitor_SMD:CP_Elec_8x10.5
Changed lines of the file:
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@@
 			)
 		)
-		(property "Footprint" "Capacitor_SMD:CP_Elec_10x7.9"
+		(property "Footprint" "Capacitor_SMD:CP_Elec_8x10.5"
 			(at 199.0852 95.25 0)
 			(effects
@@
 			)
 		)
-		(property "Footprint" "Capacitor_SMD:CP_Elec_10x7.9"
+		(property "Footprint" "Capacitor_SMD:CP_Elec_8x10.5"
 			(at 309.5752 148.59 0)
 			(effects
@@
 			)
 		)
-		(property "Footprint" "Capacitor_SMD:CP_Elec_10x7.9"
+		(property "Footprint" "Capacitor_SMD:CP_Elec_8x10.5"
 			(at 199.0852 148.59 0)
 			(effects
@@
 			)
 		)
-		(property "Footprint" "Capacitor_SMD:CP_Elec_10x7.9"
+		(property "Footprint" "Capacitor_SMD:CP_Elec_8x10.5"
 			(at 200.3552 41.91 0)
 			(effects
@@
 			)
 		)
-		(property "Footprint" "Capacitor_SMD:CP_Elec_10x7.9"
+		(property "Footprint" "Capacitor_SMD:CP_Elec_8x10.5"
 			(at 309.5752 95.25 0)
 			(effects
@@
 			)
 		)
-		(property "Footprint" "Capacitor_SMD:CP_Elec_10x7.9"
+		(property "Footprint" "Capacitor_SMD:CP_Elec_8x10.5"
 			(at 309.5752 41.91 0)
 			(effects
